File: avionics/avionics_rev1/MCU.kicad_sch (KiCad schematic)
At the start: 12 parts, among them U2 STM32G474RETx

Commit message: flight computer schematics work + 1 stage simulation
Connections:
- net GND: now also U2.29 (VDDA); no longer U2.15 (VSS), U2.27 (VSSA)
- net at C12.1, C13.1, FB2.2: no longer U2.28 (VREF+)
- net UART_TX: now reaches U2.22 (PC4)
- net UART_RX: now reaches U2.23 (PC5)
- net at FB1.2: no longer U2.29 (VDDA)
- net at U2.31 (VSS), U2.47 (VSS), U2.63 (VSS): now also U2.15 (VSS)
Other:
- note added: "TODO: pins for SPI / I2C devices pins for buzzer / status LED(s) pins for pyro channels pins for battery monitoring / current draw fix symbol power connections"
- note removed: "TODO: pins for SPI / I2C devices pins for buzzer / status LED(s) pins for pyro channels pins for battery monitoring / current draw"
- moved on the sheet: U2
Changed lines of the file:
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@@
 		)
 	)
-	(text "TODO: \npins for SPI / I2C devices\npins for buzzer / status LED(s)\npins for pyro channels\npins for battery monitoring / current draw\n\n"
+	(text "TODO: \npins for SPI / I2C devices\npins for buzzer / status LED(s)\npins for pyro channels\npins for battery monitoring / current draw\nfix symbol power connections\n"
 		(exclude_from_sim no)
 		(at 71.628 60.96 0)
@@
 	(wire
 		(pts
+			(xy 156.21 92.71) (xy 160.02 92.71)
+		)
+		(stroke
+			(width 0)
+			(type default)
+		)
+	)
+	(wire
+		(pts
 			(xy 186.69 43.18) (xy 194.31 43.18)
 		)
@@
 	(wire
 		(pts
+			(xy 156.21 95.25) (xy 160.02 95.25)
+		)
+		(stroke
+			(width 0)
+			(type default)
+		)
+	)
+	(wire
+		(pts
 			(xy 173.99 140.97) (xy 182.88 140.97)
 		)
@@
 			(width 0)
 			(type default)
+		)
+	)
+	(global_label "UART_RX"
+		(shape input)
+		(at 160.02 92.71 0)
+		(fields_autoplaced yes)
+		(effects
+			(font
+				(size 1.27 1.27)
+			)
+			(justify left)
+		)
+		(property "Intersheetrefs" "${INTERSHEET_REFS}"
+			(at 171.109 92.71 0)
+			(hide yes)
+			(show_name no)
+			(do_not_autoplace no)
+			(effects
+				(font
+					(size 1.27 1.27)
+				)
+				(justify left)
+			)
+		)
+	)
+	(global_label "UART_TX"
+		(shape input)
+		(at 160.02 95.25 0)
+		(fields_autoplaced yes)
+		(effects
+			(font
+				(size 1.27 1.27)
+			)
+			(justify left)
+		)
+		(property "Intersheetrefs" "${INTERSHEET_REFS}"
+			(at 170.8066 95.25 0)
+			(hide yes)
+			(show_name no)
+			(do_not_autoplace no)
+			(effects
+				(font
+					(size 1.27 1.27)
+				)
+				(justify left)
+			)
+		)
+	)
+	(global_label "CS_BARO"
+		(shape input)
+		(at 93.98 105.41 180)
+		(fields_autoplaced yes)
+		(effects
+			(font
+				(size 1.27 1.27)
+			)
+			(justify right)
+		)
+		(property "Intersheetrefs" "${INTERSHEET_REFS}"
+			(at 82.5886 105.41 0)
+			(hide yes)
+			(show_name no)
+			(do_not_autoplace no)
+			(effects
+				(font
+					(size 1.27 1.27)
+				)
+				(justify right)
+			)
+		)
+	)
+	(global_label "CS_IMU"
+		(shape input)
+		(at 92.71 97.79 180)
+		(fields_autoplaced yes)
+		(effects
+			(font
+				(size 1.27 1.27)
+			)
+			(justify right)
+		)
+		(property "Intersheetrefs" "${INTERSHEET_REFS}"
+			(at 82.891 97.79 0)
+			(hide yes)
+			(show_name no)
+			(do_not_autoplace no)
+			(effects
+				(font
+					(size 1.27 1.27)
+				)
+				(justify right)
+			)
 		)
 	)
@@
 			(hide yes)
 			(show_name no)
+			(do_not_autoplace no)
+			(effects
+				(font
+					(size 1.27 1.27)
+				)
+				(justify right)
+			)
+		)
+	)
+	(global_label "GPS_RESET"
+		(shape input)
+		(at 93.98 92.71 180)
+		(fields_autoplaced yes)
+		(effects
+			(font
+				(size 1.27 1.27)
+			)
+			(justify right)
+		)
+		(property "Intersheetrefs" "${INTERSHEET_REFS}"
+			(at 80.5326 92.71 0)
+			(hide yes)
+			(show_name no)

Commit message: more avionics work
Parts:
- removed C12: 1uF, Capacitor_SMD:C_0201_0603Metric, symbol Device:C_Small
- added BZ1: Buzzer, avionics_footprints:XDCR_PS1240P02BT, symbol Device:Buzzer
- added C15: 1uF, Capacitor_SMD:C_0201_0603Metric, symbol Device:C_Small
Connections:
- net GND: now also U2.15 (VSS), U2.27 (VSSA), U2.31 (VSS), U2.47 (VSS), U2.63 (VSS), C15.2; no longer U2.29 (VDDA)
- net VREF: now reaches C13.1, FB2.2
- net VREF: now also U2.28 (VREF+), C15.1
- net at FB1.2: now also U2.29 (VDDA)
Other:
- note added: "TODO: pins for SPI / I2C devices pins for buzzer / status LED(s) pins for pyro channels pins for battery monitoring / current draw"
- note removed: "TODO: pins for SPI / I2C devices pins for buzzer / status LED(s) pins for pyro channels pins for battery monitoring / current draw fix symbol power connections"
- moved on the sheet: C13
