File: avionics/avionics_rev1/MCU.kicad_sch (KiCad schematic)
At the start: 40 parts, among them J5 FTSH-107-01-L-DV-K, Q2 DMN2056U-7, U14 W25Q512JVFIM, U2 STM32G474RET6, Y1 16MHz / CL10pF

Commit message: adjusted resistor footprints to 0603
Parts:
- R46, R47, R48, R49, R50, R54, R55, R56, R57, R58, R59, R60: footprint Resistor_SMD:R_0402_1005Metric -> Resistor_SMD:R_0603_1608Metric
Changed lines of the file:
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@@
 		(dnp no)
 		(property "Reference" "Q2"
-			(at 353.695 48.26 0)
+			(at 349.758 48.006 0)
 			(show_name no)
 			(do_not_autoplace no)
@@
 		)
 		(property "Value" "DMN2056U-7"
-			(at 353.695 50.8 0)
+			(at 349.758 50.546 0)
 			(show_name no)
 			(do_not_autoplace no)
@@
 		(dnp no)
 		(property "Reference" "R56"
-			(at 327.66 33.02 0)
+			(at 332.74 32.258 0)
 			(show_name no)
 			(do_not_autoplace no)
@@
 		)
 		(property "Value" "1k"
-			(at 327.66 35.56 0)
+			(at 332.74 34.29 0)
 			(show_name no)
 			(do_not_autoplace no)
@@
 			)
 		)
-		(property "Footprint" "Resistor_SMD:R_0402_1005Metric"
+		(property "Footprint" "Resistor_SMD:R_0603_1608Metric"
 			(at 336.55 34.29 0)
 			(hide yes)
@@
 		)
 		(property "Tolerance" "1%"
-			(at 327.66 37.46 0)
+			(at 332.74 36.19 0)
 			(show_name no)
 			(do_not_autoplace yes)
@@
 			)
 		)
-		(property "Footprint" "Resistor_SMD:R_0402_1005Metric"
+		(property "Footprint" "Resistor_SMD:R_0603_1608Metric"
 			(at 306.07 109.22 0)
 			(hide yes)
@@
 			)
 		)
-		(property "Footprint" "Resistor_SMD:R_0402_1005Metric"
+		(property "Footprint" "Resistor_SMD:R_0603_1608Metric"
 			(at 45.72 101.6 0)
 			(hide yes)
@@
 		(dnp no)
 		(property "Reference" "R54"
-			(at 316.23 43.18 90)
+			(at 316.23 44.196 90)
 			(show_name no)
 			(do_not_autoplace no)
@@
 			)
 		)
-		(property "Footprint" "Resistor_SMD:R_0402_1005Metric"
+		(property "Footprint" "Resistor_SMD:R_0603_1608Metric"
 			(at 316.23 49.53 0)
 			(hide yes)
@@
 		)
 		(property "Tolerance" "1%"
-			(at 316.23 47.62 0)
+			(at 316.23 47.498 90)
 			(show_name no)
 			(do_not_autoplace yes)
@@
 			)
 		)
-		(property "Footprint" "Resistor_SMD:R_0402_1005Metric"
+		(property "Footprint" "Resistor_SMD:R_0603_1608Metric"
 			(at 106.68 204.47 0)
 			(hide yes)
@@
 			)
 		)
-		(property "Footprint" "Resistor_SMD:R_0402_1005Metric"
+		(property "Footprint" "Resistor_SMD:R_0603_1608Metric"
 			(at 228.6 104.14 0)
 			(hide yes)
@@
 			)
 		)
-		(property "Footprint" "Resistor_SMD:R_0402_1005Metric"
+		(property "Footprint" "Resistor_SMD:R_0603_1608Metric"
 			(at 36.83 101.6 0)
 			(hide yes)
@@
 			)
 		)
-		(property "Footprint" "Resistor_SMD:R_0402_1005Metric"
+		(property "Footprint" "Resistor_SMD:R_0603_1608Metric"
 			(at 54.61 101.6 0)
 			(hide yes)
@@
 		(in_pos_files yes)
 		(dnp no)
-		(fields_autoplaced yes)
 		(property "Reference" "R50"
 			(at 143.51 93.98 90)
@@
 			)
 		)
-		(property "Footprint" "Resistor_SMD:R_0402_1005Metric"
+		(property "Footprint" "Resistor_SMD:R_0603_1608Metric"
 			(at 143.51 100.33 0)
 			(hide yes)
@@
 		)
 		(property "Tolerance" "1%"
-			(at 143.51 98.42 0)
+			(at 143.51 98.298 90)
 			(show_name no)
 			(do_not_autoplace yes)
@@
 		(dnp no)
 		(property "Reference" "BZ1"
-			(at 349.25 22.86 0)
+			(at 357.886 32.512 0)
 			(show_name no)
 			(do_not_autoplace no)
@@
 		)
 		(property "Value" "PS1240P02BT"
-			(at 349.25 25.4 0)
+			(at 357.886 35.052 0)
 			(show_name no)
 			(do_not_autoplace no)
@@
 			)
 		)
-		(property "Footprint" "Resistor_SMD:R_0402_1005Metric"
+		(property "Footprint" "Resistor_SMD:R_0603_1608Metric"
 			(at 290.83 104.14 0)
 			(hide yes)
@@
 		(dnp no)
 		(property "Reference" "R55"
-			(at 316.23 58.42 0)
+			(at 324.866 58.166 0)
 			(show_name no)
 			(do_not_autoplace no)
@@
 		)
 		(property "Value" "10k"
-			(at 316.23 60.96 0)
+			(at 324.866 59.944 0)
 			(show_name no)
 			(do_not_autoplace no)
@@
 			)
 		)
-		(property "Footprint" "Resistor_SMD:R_0402_1005Metric"
+		(property "Footprint" "Resistor_SMD:R_0603_1608Metric"
 			(at 328.93 59.69 0)
 			(hide yes)
@@
 		)
 		(property "Tolerance" "1%"
-			(at 316.23 62.86 0)
+			(at 324.866 61.844 0)
 			(show_name no)
 			(do_not_autoplace yes)
@@
 			)
 		)
-		(property "Footprint" "Resistor_SMD:R_0402_1005Metric"
+		(property "Footprint" "Resistor_SMD:R_0603_1608Metric"
 			(at 63.5 101.6 0)
 			(hide yes)

Commit message: finished updating footprints
Parts:
- C10, C11, C42, C43, C52: Manufacturer (none) -> TDK
- C14, C41, C44, C51, C6, C7, C8, C9: footprint Capacitor_SMD:C_0402_1005Metric -> Capacitor_SMD:C_0603_1608Metric; DigiKey https://www.digikey.com/en/products/detail/murata-electroni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 -> https://www.digikey.com/en/products/detail/kemet/C0603C104K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; MPN GRM155R71A104KA01D -> C0603C104K5RACTU; Manufacturer (none) -> KEMET; Voltage 10V -> 50V
- C39, C40: footprint Capacitor_SMD:C_0402_1005Metric -> Capacitor_SMD:C_0603_1608Metric; DigiKey https://www.digikey.com/en/products/detail/kemet/C0402C100J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 -> https://www.digikey.com/en/products/detail/kemet/C0603C100J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; MPN C0402C100J5GACTU -> C0603C100J5GACTU; Manufacturer (none) -> KEMET
- R46, R47, R48, R49, R55, R57, R58, R59, R60: DigiKey https://www.digikey.com/en/products/detail/yageo/RC0402FR-0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 -> https://www.digikey.com/en/products/detail/yageo/RC0603FR-0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; MPN RC0402FR-0710KL -> RC0603FR-0710KL; Manufacturer (none) -> Yageo; Power (none) -> 0.1W; Voltage 50V -> 75V
- R50, R54, R56: DigiKey https://www.digikey.com/en/products/detail/yageo/RC0402FR-0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 -> https://www.digikey.com/en/products/detail/yageo/RC0603FR-0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; MPN RC0402FR-071KL -> RC0603FR-071KL; Manufacturer (none) -> Yageo; Power 0.063W -> 0.1W; Voltage 50V -> 75V

Commit message: layout 1
Parts:
- C11, C51, C52, FB2, TP10, TP11, TP12, TP13: now not fitted
Connections:
- net VREF_FILTERED is gone; now on net VDDA_FILTERED: C51.1, C52.1, FB2.2, U2.28 (VREF+)
Changed lines of the file:
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@@
 	)
 	(junction
+		(at 64.77 181.61)
+		(diameter 0)
+		(color 0 0 0 0)
+	)
+	(junction
 		(at 52.07 85.09)
 		(diameter 0)
@@
 	(wire
 		(pts
+			(xy 66.04 179.07) (xy 64.77 179.07)
+		)
+		(stroke
+			(width 0)
+			(type default)
+		)
+	)
+	(wire
+		(pts
 			(xy 33.02 181.61) (xy 25.4 181.61)
 		)
@@
 	(wire
 		(pts
+			(xy 64.77 179.07) (xy 64.77 181.61)
+		)
+		(stroke
+			(width 0)
+			(type default)
+		)
+	)
+	(wire
+		(pts
 			(xy 85.09 72.39) (xy 81.28 72.39)
 		)
@@
 	(wire
 		(pts
-			(xy 59.69 181.61) (xy 66.04 181.61)
+			(xy 59.69 181.61) (xy 64.77 181.61)
 		)
 		(stroke
@@
 	(wire
 		(pts
+			(xy 64.77 181.61) (xy 66.04 181.61)
+		)
+		(stroke
+			(width 0)
+			(type default)
+		)
+	)
+	(wire
+		(pts
 			(xy 217.17 39.37) (xy 212.09 39.37)
 		)
@@
 		)
 	)
+	(label "VREF_FILTERED"
+		(at 66.04 179.07 0)
+		(effects
+			(font
+				(size 1 1)
+			)
+			(justify left bottom)
+		)
+	)
 	(label "BUZZER_PWM"
 		(at 125.73 97.79 0)
@@
 		(exclude_from_sim no)
 		(in_bom no)
-		(on_board yes)
+		(on_board no)
 		(in_pos_files yes)
-		(dnp no)
+		(dnp yes)
 		(property "Reference" "TP13"
 			(at 61.976 93.98 0)
@@
 		(exclude_from_sim no)
 		(in_bom no)
-		(on_board yes)
+		(on_board no)
 		(in_pos_files yes)
-		(dnp no)
+		(dnp yes)
 		(property "Reference" "TP12"
 			(at 53.086 93.98 0)
@@
 		(exclude_from_sim no)
 		(in_bom yes)
-		(on_board yes)
+		(on_board no)
 		(in_pos_files yes)
-		(dnp no)
+		(dnp yes)
 		(property "Reference" "C51"
 			(at 50.8 204.47 0)
@@
 		(exclude_from_sim no)
 		(in_bom yes)
-		(on_board yes)
+		(on_board no)
 		(in_pos_files yes)
-		(dnp no)
+		(dnp yes)
 		(property "Reference" "C52"
 			(at 66.04 204.47 0)
@@
 		(on_board yes)
 		(in_pos_files yes)
-		(dnp no)
+		(dnp yes)
 		(property "Reference" "C11"
 			(at 113.792 162.56 0)
@@
 		(exclude_from_sim no)
 		(in_bom yes)
-		(on_board yes)
+		(on_board no)
 		(in_pos_files yes)
-		(dnp no)
+		(dnp yes)
 		(property "Reference" "FB2"
 			(at 36.068 195.834 90)
@@
 		(exclude_from_sim no)
 		(in_bom no)
-		(on_board yes)
+		(on_board no)
 		(in_pos_files yes)
-		(dnp no)
+		(dnp yes)
 		(property "Reference" "TP10"
 			(at 35.306 93.98 0)
@@
 		(exclude_from_sim no)
 		(in_bom no)
-		(on_board yes)
+		(on_board no)
 		(in_pos_files yes)
-		(dnp no)
+		(dnp yes)
 		(property "Reference" "TP11"
 			(at 44.196 93.98 0)
