File: avionics/avionics_rev1/avionics_rev1.kicad_sch (KiCad schematic)
At the start: 0 parts

Commit message: flight computer schematics work + 1 stage simulation
Other:
- added sheet GPS (GPS.kicad_sch)
- added sheet IMU (IMU.kicad_sch)
- added sheet Radio (Radio.kicad_sch)
- added sheet barometer (barometer.kicad_sch)
- note added: "LPS22DF datasheet: https://www.st.com/resource/en/datasheet/lps22df.pdf"
- note added: "LSM6DSV32X datasheet: https://www.st.com/resource/en/datasheet/lsm6dsv32x.pdf"
- note added: "MAX-M10S-00B datasheet: https://content.u-blox.com/sites/default/files/MAX-M10S_DataSheet_UBX-20035208.pdf"
- note added: "Wio-SX1262 datasheet: https://files.seeedstudio.com/products/SenseCAP/Wio_SX1262/Wio-SX1262_Module_Datasheet.pdf"
Changed lines of the file:
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@@
 	(generator_version "10.0")
 	(paper "A4")
+	(text "LPS22DF datasheet:\nhttps://www.st.com/resource/en/datasheet/lps22df.pdf"
+		(exclude_from_sim no)
+		(at 26.67 98.806 0)
+		(effects
+			(font
+				(size 1.27 1.27)
+			)
+			(justify left)
+		)
+	)
+	(text "Wio-SX1262 datasheet:\nhttps://files.seeedstudio.com/products/SenseCAP/Wio_SX1262/Wio-SX1262_Module_Datasheet.pdf"
+		(exclude_from_sim no)
+		(at 30.988 147.574 0)
+		(effects
+			(font
+				(size 1.27 1.27)
+			)
+			(justify left)
+		)
+	)
+	(text "LSM6DSV32X datasheet:\nhttps://www.st.com/resource/en/datasheet/lsm6dsv32x.pdf"
+		(exclude_from_sim no)
+		(at 25.654 75.692 0)
+		(effects
+			(font
+				(size 1.27 1.27)
+			)
+			(justify left)
+		)
+	)
 	(text "STM32G474RET6 datasheet:\nhttps://www.st.com/resource/en/datasheet/stm32g474cb.pdf"
 		(exclude_from_sim no)
 		(at 23.876 40.386 0)
+		(effects
+			(font
+				(size 1.27 1.27)
+			)
+			(justify left)
+		)
+	)
+	(text "MAX-M10S-00B datasheet:\nhttps://content.u-blox.com/sites/default/files/MAX-M10S_DataSheet_UBX-20035208.pdf"
+		(exclude_from_sim no)
+		(at 30.226 123.19 0)
 		(effects
 			(font
@@
 	)
 	(sheet
+		(at 24.13 68.58)
+		(size 62.23 13.97)
+		(exclude_from_sim no)
+		(in_bom yes)
+		(on_board yes)
+		(dnp no)
+		(fields_autoplaced yes)
+		(stroke
+			(width 0.1524)
+			(type solid)
+		)
+		(fill
+			(color 0 0 0 0)
+		)
+		(property "Sheetname" "IMU"
+			(at 24.13 67.8684 0)
+			(show_name no)
+			(do_not_autoplace no)
+			(effects
+				(font
+					(size 1.27 1.27)
+				)
+				(justify left bottom)
+			)
+		)
+		(property "Sheetfile" "IMU.kicad_sch"
+			(at 24.13 83.1346 0)
+			(show_name no)
+			(do_not_autoplace no)
+			(effects
+				(font
+					(size 1.27 1.27)
+				)
+				(justify left top)
+			)
+		)
+		(instances
+			(project "avionics_rev1"
+				(path "/c491fe45-d2ff-414d-a846-7eed12d2b763"
+					(page "5")
+				)
+			)
+		)
+	)
+	(sheet
+		(at 27.94 115.57)
+		(size 93.98 15.24)
+		(exclude_from_sim no)
+		(in_bom yes)
+		(on_board yes)
+		(dnp no)
+		(fields_autoplaced yes)
+		(stroke
+			(width 0.1524)
+			(type solid)
+		)
+		(fill
+			(color 0 0 0 0)
+		)
+		(property "Sheetname" "GPS"
+			(at 27.94 114.8584 0)
+			(show_name no)
+			(do_not_autoplace no)
+			(effects
+				(font
+					(size 1.27 1.27)
+				)
+				(justify left bottom)
+			)
+		)
+		(property "Sheetfile" "GPS.kicad_sch"
+			(at 27.94 131.3946 0)
+			(show_name no)
+			(do_not_autoplace no)
+			(effects
+				(font
+					(size 1.27 1.27)
+				)
+				(justify left top)
+			)
+		)
+		(instances
+			(project "avionics_rev1"
+				(path "/c491fe45-d2ff-414d-a846-7eed12d2b763"
+					(page "7")
+				)
+			)
+		)
+	)
+	(sheet
+		(at 29.21 143.51)
+		(size 100.33 8.89)
+		(exclude_from_sim no)
+		(in_bom yes)
+		(on_board yes)
+		(dnp no)
+		(fields_autoplaced yes)
+		(stroke
+			(width 0.1524)
+			(type solid)
+		)
+		(fill
+			(color 0 0 0 0)
+		)
+		(property "Sheetname" "Radio"
+			(at 29.21 142.7984 0)
+			(show_name no)
+			(do_not_autoplace no)
+			(effects
+				(font
+					(size 1.27 1.27)
+				)
+				(justify left bottom)
+			)
+		)
+		(property "Sheetfile" "Radio.kicad_sch"
+			(at 29.21 152.9846 0)
+			(show_name no)
+			(do_not_autoplace no)
+			(effects
+				(font
+					(size 1.27 1.27)
+				)
+				(justify left top)
+			)
+		)
+		(instances
+			(project "avionics_rev1"
+				(path "/c491fe45-d2ff-414d-a846-7eed12d2b763"
+					(page "8")
+				)
+			)
+		)
+	)
+	(sheet
 		(at 22.86 48.26)
 		(size 91.44 10.16)
@@
 				)
 			)
+		)
+	)
+	(sheet
+		(at 24.13 91.44)
+		(size 60.96 16.51)
+		(exclude_from_sim no)
+		(in_bom yes)
+		(on_board yes)
+		(dnp no)
+		(fields_autoplaced yes)
+		(stroke
+			(width 0.1524)
+			(type solid)
+		)
+		(fill
+			(color 0 0 0 0)
+		)
+		(property "Sheetname" "barometer"
+			(at 24.13 90.7284 0)
+			(show_name no)
+			(do_not_autoplace no)
+			(effects
+				(font
+					(size 1.27 1.27)
+				)
+				(justify left bottom)
+			)
+		)
+		(property "Sheetfile" "barometer.kicad_sch"
+			(at 24.13 108.5346 0)
+			(show_name no)
+			(do_not_autoplace no)
+			(effects
+				(font
+					(size 1.27 1.27)
+				)
+				(justify left top)
+			)
+		)
+		(instances
+			(project "avionics_rev1"
+				(path "/c491fe45-d2ff-414d-a846-7eed12d2b763"
+					(page "6")
+				)
+			)

Commit message: more avionics work
Other:
- removed sheet GPS
- removed sheet IMU
- removed sheet Radio
- removed sheet accelerometer
- removed sheet barometer
- added sheet sensors (sensors.kicad_sch)
- added sheet telemetry (telemetry.kicad_sch)
- note removed: "ADXL375BCCZ-RL7 datasheet: https://www.analog.com/media/en/technical-documentation/data-sheets/ADXL375.pdf"
- note removed: "LPS22DF datasheet: https://www.st.com/resource/en/datasheet/lps22df.pdf"
- note removed: "LSM6DSV32X datasheet: https://www.st.com/resource/en/datasheet/lsm6dsv32x.pdf"
- note removed: "MAX-M10S-00B datasheet: https://content.u-blox.com/sites/default/files/MAX-M10S_DataSheet_UBX-20035208.pdf"
Changed lines of the file:
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@@
 	(generator_version "10.0")
 	(paper "A4")
-	(text "LPS22DF datasheet:\nhttps://www.st.com/resource/en/datasheet/lps22df.pdf"
-		(exclude_from_sim no)
-		(at 26.67 98.806 0)
-		(effects
-			(font
-				(size 1.27 1.27)
-			)
-			(justify left)
-		)
-	)
 	(text "Wio-SX1262 datasheet:\nhttps://files.seeedstudio.com/products/SenseCAP/Wio_SX1262/Wio-SX1262_Module_Datasheet.pdf"
 		(exclude_from_sim no)
 		(at 30.988 147.574 0)
-		(effects
-			(font
-				(size 1.27 1.27)
-			)
-			(justify left)
-		)
-	)
-	(text "LSM6DSV32X datasheet:\nhttps://www.st.com/resource/en/datasheet/lsm6dsv32x.pdf"
-		(exclude_from_sim no)
-		(at 25.654 75.692 0)
 		(effects
 			(font
@@
 		)
 	)
-	(text "MAX-M10S-00B datasheet:\nhttps://content.u-blox.com/sites/default/files/MAX-M10S_DataSheet_UBX-20035208.pdf"
-		(exclude_from_sim no)
-		(at 30.226 123.19 0)
-		(effects
-			(font
-				(size 1.27 1.27)
-			)
-			(justify left)
-		)
-	)
 	(text "LMR604063SBRAKRQ1 datasheet:\nhttps://www.ti.com/lit/ds/symlink/lmr60406-q1.pdf"
 		(exclude_from_sim no)
 		(at 24.13 26.924 0)
-		(effects
-			(font
-				(size 1.27 1.27)
-			)
-			(justify left)
-		)
-	)
-	(text "ADXL375BCCZ-RL7 datasheet:\nhttps://www.analog.com/media/en/technical-documentation/data-sheets/ADXL375.pdf"
-		(exclude_from_sim no)
-		(at 24.892 53.34 0)
 		(effects
 			(font
@@
 	)
 	(sheet
-		(at 24.13 68.58)
-		(size 62.23 13.97)
+		(at 38.1 63.5)
+		(size 35.56 11.43)
 		(exclude_from_sim no)
 		(in_bom yes)
@@
 			(color 0 0 0 0)
 		)
-		(property "Sheetname" "IMU"
-			(at 24.13 67.8684 0)
+		(property "Sheetname" "telemetry"
+			(at 38.1 62.7884 0)
 			(show_name no)
 			(do_not_autoplace no)
@@
 			)
 		)
-		(property "Sheetfile" "IMU.kicad_sch"
-			(at 24.13 83.1346 0)
+		(property "Sheetfile" "telemetry.kicad_sch"
+			(at 38.1 75.5146 0)
+			(show_name no)
+			(do_not_autoplace no)
+			(effects
+				(font
+					(size 1.27 1.27)
+				)
+				(justify left top)
+			)
+		)
+		(instances
+			(project "avionics_rev1"
+				(path "/c491fe45-d2ff-414d-a846-7eed12d2b763"
+					(page "4")
+				)
+			)
+		)
+	)
+	(sheet
+		(at 140.97 57.15)
+		(size 12.7 3.81)
+		(exclude_from_sim no)
+		(in_bom yes)
+		(on_board yes)
+		(dnp no)
+		(fields_autoplaced yes)
+		(stroke
+			(width 0.1524)
+			(type solid)
+		)
+		(fill
+			(color 0 0 0 0)
+		)
+		(property "Sheetname" "sensors"
+			(at 140.97 56.4384 0)
+			(show_name no)
+			(do_not_autoplace no)
+			(effects
+				(font
+					(size 1.27 1.27)
+				)
+				(justify left bottom)
+			)
+		)
+		(property "Sheetfile" "sensors.kicad_sch"
+			(at 140.97 61.5446 0)
 			(show_name no)
 			(do_not_autoplace no)
@@
 				)
 			)
-		)
-	)
-	(sheet
-		(at 27.94 115.57)
-		(size 93.98 15.24)
-		(exclude_from_sim no)
-		(in_bom yes)
-		(on_board yes)
-		(dnp no)
-		(fields_autoplaced yes)
-		(stroke
-			(width 0.1524)
-			(type solid)
-		)
-		(fill
-			(color 0 0 0 0)
-		)
-		(property "Sheetname" "GPS"
-			(at 27.94 114.8584 0)
-			(show_name no)
-			(do_not_autoplace no)
-			(effects
-				(font
-					(size 1.27 1.27)
-				)
-				(justify left bottom)
-			)
-		)
-		(property "Sheetfile" "GPS.kicad_sch"
-			(at 27.94 131.3946 0)
-			(show_name no)
-			(do_not_autoplace no)
-			(effects
-				(font
-					(size 1.27 1.27)
-				)
-				(justify left top)
-			)
-		)
-		(instances
-			(project "avionics_rev1"
-				(path "/c491fe45-d2ff-414d-a846-7eed12d2b763"
-					(page "7")
-				)
-			)
-		)
-	)
-	(sheet
-		(at 29.21 143.51)
-		(size 100.33 8.89)
-		(exclude_from_sim no)
-		(in_bom yes)
-		(on_board yes)
-		(dnp no)
-		(fields_autoplaced yes)
-		(stroke
-			(width 0.1524)
-			(type solid)
-		)
-		(fill
-			(color 0 0 0 0)
-		)
-		(property "Sheetname" "Radio"
-			(at 29.21 142.7984 0)
-			(show_name no)
-			(do_not_autoplace no)
-			(effects
-				(font
-					(size 1.27 1.27)
-				)
-				(justify left bottom)
-			)
-		)
-		(property "Sheetfile" "Radio.kicad_sch"
-			(at 29.21 152.9846 0)
-			(show_name no)
-			(do_not_autoplace no)
-			(effects
-				(font
-					(size 1.27 1.27)
-				)
-				(justify left top)
-			)
-		)
-		(instances
-			(project "avionics_rev1"
-				(path "/c491fe45-d2ff-414d-a846-7eed12d2b763"
-					(page "8")
-				)
-			)
-		)
-	)
-	(sheet
-		(at 22.86 48.26)
-		(size 91.44 10.16)
-		(exclude_from_sim no)
-		(in_bom yes)
-		(on_board yes)
-		(dnp no)
-		(fields_autoplaced yes)
-		(stroke
-			(width 0.1524)
-			(type solid)
-		)
-		(fill
-			(color 0 0 0 0)
-		)
-		(property "Sheetname" "accelerometer"
-			(at 22.86 47.5484 0)
-			(show_name no)
-			(do_not_autoplace no)
-			(effects
-				(font
-					(size 1.27 1.27)
-				)
-				(justify left bottom)
-			)
-		)
-		(property "Sheetfile" "accelerometer.kicad_sch"
-			(at 22.86 59.0046 0)
-			(show_name no)
-			(do_not_autoplace no)
-			(effects
-				(font
-					(size 1.27 1.27)
-				)
-				(justify left top)
-			)
-		)
-		(property "Field2" ""
-			(at 22.86 48.26 0)
-			(hide yes)
-			(show_name no)
-			(do_not_autoplace no)
-			(effects
-				(font
-					(size 1.27 1.27)
-				)
-			)
-		)
-		(instances
-			(project "avionics_rev1"
-				(path "/c491fe45-d2ff-414d-a846-7eed12d2b763"
-					(page "4")
-				)
-			)
-		)
-	)
-	(sheet
-		(at 24.13 91.44)
-		(size 60.96 16.51)
-		(exclude_from_sim no)
-		(in_bom yes)
-		(on_board yes)
-		(dnp no)
-		(fields_autoplaced yes)
-		(stroke
-			(width 0.1524)
-			(type solid)
-		)
-		(fill
-			(color 0 0 0 0)
-		)
-		(property "Sheetname" "barometer"
-			(at 24.13 90.7284 0)
-			(show_name no)
-			(do_not_autoplace no)
-			(effects
-				(font
-					(size 1.27 1.27)
-				)
-				(justify left bottom)
-			)
-		)
-		(property "Sheetfile" "barometer.kicad_sch"
-			(at 24.13 108.5346 0)
-			(show_name no)
-			(do_not_autoplace no)
-			(effects
-				(font
-					(size 1.27 1.27)
-				)
-				(justify left top)
-			)
-		)
-		(instances
-			(project "avionics_rev1"
-				(path "/c491fe45-d2ff-414d-a846-7eed12d2b763"
-					(page "6")
-				)
-			)
