File: avionics/avionics_rev1/avionics_rev1.kicad_sch (KiCad schematic)
At the start: 0 parts

Commit message: saving work before chat
Other:
- added sheet pyro_channels (pyro_channels.kicad_sch)
Changed lines of the file:
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@@
+	)
+	(sheet
+		(at 130.81 96.52)
+		(size 27.94 11.43)
+		(exclude_from_sim no)
+		(in_bom yes)
+		(on_board yes)
+		(dnp no)
+		(fields_autoplaced yes)
+		(stroke
+			(width 0.1524)
+			(type solid)
+		)
+		(fill
+			(color 0 0 0 0)
+		)
+		(property "Sheetname" "pyro_channels"
+			(at 130.81 95.8084 0)
+			(show_name no)
+			(do_not_autoplace no)
+			(effects
+				(font
+					(size 1.27 1.27)
+				)
+				(justify left bottom)
+			)
+		)
+		(property "Sheetfile" "pyro_channels.kicad_sch"
+			(at 130.81 108.5346 0)
+			(show_name no)
+			(do_not_autoplace no)
+			(effects
+				(font
+					(size 1.27 1.27)
+				)
+				(justify left top)
+			)
+		)
+		(instances
+			(project "avionics_rev1"
+				(path "/c491fe45-d2ff-414d-a846-7eed12d2b763"
+					(page "6")
+				)
+			)
+		)
 	)
 	(sheet

Commit message: working on sensors schematics
Other:
- note added: "TODO: Draw system schematic with relevant sheets at a high level Consolidate datasheets to their respective sheets/parts Write specs/assumptions on this page Find a flash chip and connect it to MCU"
- note removed: "TODO: consolidate sensors into 1 sheet if needed"
Changed lines of the file:
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@@
 		)
 	)
-	(text "TODO: consolidate sensors into 1 sheet if needed"
+	(text "TODO:\nDraw system schematic with relevant sheets at a high level\nConsolidate datasheets to their respective sheets/parts\nWrite specs/assumptions on this page\nFind a flash chip and connect it to MCU"
 		(exclude_from_sim no)
-		(at 218.948 33.782 0)
+		(at 41.148 114.046 0)
 		(effects
 			(font
-				(size 1.27 1.27)
+				(size 2.032 2.032)
+				(thickness 0.254)
+				(bold yes)
 			)
 			(justify left)
@@
 	)
 	(sheet
-		(at 130.81 96.52)
+		(at 139.7 86.36)
 		(size 27.94 11.43)
 		(exclude_from_sim no)
@@
 		)
 		(property "Sheetname" "pyro_channels"
-			(at 130.81 95.8084 0)
+			(at 139.7 85.6484 0)
 			(show_name no)
 			(do_not_autoplace no)
@@
 		)
 		(property "Sheetfile" "pyro_channels.kicad_sch"
-			(at 130.81 108.5346 0)
+			(at 139.7 98.3746 0)
 			(show_name no)
 			(do_not_autoplace no)

Commit message: cleaned up schematics after codex work
Other:
- note added: "TODO: Draw system schematic with relevant sheets at a high level Consolidate datasheets to their respective sheets/parts Write specs/assumptions on this page Put test pads everywhere!"
- note removed: "TODO: Draw system schematic with relevant sheets at a high level Consolidate datasheets to their respective sheets/parts Write specs/assumptions on this page Find a flash chip and connect it to MCU"
Changed lines of the file:
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@@
 		)
 	)
-	(text "TODO:\nDraw system schematic with relevant sheets at a high level\nConsolidate datasheets to their respective sheets/parts\nWrite specs/assumptions on this page\nFind a flash chip and connect it to MCU"
+	(text "TODO:\nDraw system schematic with relevant sheets at a high level\nConsolidate datasheets to their respective sheets/parts\nWrite specs/assumptions on this page\nPut test pads everywhere!"
 		(exclude_from_sim no)
 		(at 41.148 114.046 0)
