File: avionics/avionics_rev1/power_setup.kicad_sch (KiCad schematic)
At the start: 13 parts, among them U1 LMR604065SRAKRQ1

Commit message: flight computer schematics work + 1 stage simulation
Parts:
- U1: footprint avionics_footprints:RAK0009A-MFG -> RAK0009A-MFG
Connections:
- net PG_SENS: no longer U1.5 (PG)
Changed lines of the file:
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@@
 			)
 		)
-		(property "Footprint" "avionics_footprints:RAK0009A-MFG"
+		(property "Footprint" "RAK0009A-MFG"
 			(at 157.226 67.31 0)
 			(hide yes)

Commit message: more avionics work
Parts:
- added J1: Conn_01x02, symbol Connector_Generic:Conn_01x02
- L1: footprint (none) -> Inductor_SMD:L_Changjiang_FTC303010D
Connections:
- net +3.3V: now also R5.1
- net PG_SENS: now also U1.5 (PG); no longer R5.1
Other:
- moved on the sheet: C1, C2, C4, C5, R1
