File: avionics/avionics_rev1/power_setup.kicad_sch (KiCad schematic)
At the start: 14 parts, among them J1 Conn_01x02, U1 LMR604065SRAKRQ1

Commit message: saving work before chat
Parts:
- added C12, C18: 0.1u, symbol Device:C_Small
- added C16, C17: 10u, symbol Device:C_Small
- added C19: 10n, symbol Device:C_Small
- added D2, D3: TODO, Diode_THT:D_DO-201AE_P15.24mm_Horizontal, symbol Diode:1N62xxCA
- added D4: BZT52Bxx, Diode_SMD:D_SOD-123F, symbol Diode:BZT52Bxx
- added J2: Conn_01x02, symbol Connector_Generic:Conn_01x02
- added J4: USB_C_Receptacle_USB2.0_16P, symbol Connector:USB_C_Receptacle_USB2.0_16P
- added Q1: DMN2056U, Package_TO_SOT_SMD:SOT-23, symbol Transistor_FET:DMN2056U
- added R19: 20k, symbol Device:R_Small_US
- added R20, R21: 5.1k, Resistor_SMD:R_0201_0603Metric, symbol Device:R_Small_US
- added R22, R24, R29, R31, R33: 10k, symbol Device:R_Small_US
- added R23: 18.2k, symbol Device:R_Small_US
- added R25, R26, R35: 47k, symbol Device:R_Small_US
- added R27: 100k, symbol Device:R_Small_US
- added R28: 1k, symbol Device:R_Small_US
- added R30, R32: 49.9k, symbol Device:R_Small_US
- added R34: 22.1k, symbol Device:R_Small_US
- added U5: TPS2121RUXR, RUX0012A, symbol rocketry_library:TPS2121RUXR
- added U6: TLV7041DBV, Package_TO_SOT_SMD:SOT-23-5, symbol Comparator:TLV7041DBV
- added U7: TMUX1511RSVR, RSV0016A-MFG, symbol rocketry_library:TMUX1511RSVR
- U1: value LMR604065SRAKRQ1 -> LMR604063SBRAKRQ1
Connections:
- net +3.3V: now also C12.1, R23.1, U6.5 (V+)
- net GND: now also J1.1 (Pin_1), C12.2, C16.2, C17.2, C18.2, C19.2, D2.1 (A1), D3.1 (A1), D4.2 (A), J2.1 (Pin_1), J4.A1 (GND), J4.A12 (GND), J4.B1 (GND), J4.B12 (GND), Q1.2 (S), R20.1, R21.1, R22.2, R24.2, R26.2, R27.2, R31.2, R33.2, R34.2, R35.2, U5.11 (SS), U5.12 (GND), U5.3 (CP2), U6.2 (V-)
- net VIN_BATT: now also J1.2 (Pin_2); no longer C1.1, C2.1, R3.2, U1.1 (VIN), U1.9 (EN)
- net PG_SENS renamed MCU_PG_SENS
- new net: D4.1 (K), Q1.3 (D), R29.1, U5.4 (OV2)
- new net: R25.2, R26.1
- new net: J4.A5 (CC1), R21.2
- new net: R34.1, U5.10 (ILM)
- new net: R23.2, R24.1, U6.3 (+)
- new net: J4.B5 (CC2), R20.2
- new net: Q1.1 (G), R27.1, R28.2
- new net: U5.5 (OV1), U6.1
- new net: R19.2, R22.1, U5.6 (PR1), U6.4 (-)
- new net MAIN_BAT_SENS: R30.2, R31.1
- new net PYRO_PMUX_ST: U5.9 (ST)
- new net PYRO_POWER: C18.1, R32.1, R35.1, U5.1 (OUT), U5.8 (OUT)
- new net PYRO_POWER_SENS: C19.1, R32.2, R33.1
- new net PYRO_SEL_IN2: R28.1
- new net USB_D+: D3.2 (A2), J4.A6 (D+), J4.B6 (D+)
- new net USB_D-: D2.2 (A2), J4.A7 (D-), J4.B7 (D-)
- new net VIN_LOGIC: C1.1, C2.1, R3.2, U1.1 (VIN), U1.9 (EN)
- new net VIN_MAIN_BATT: C16.1, R29.2, R30.1, U5.2 (IN2)
- new net VIN_PYRO_BATT: C17.1, J2.2 (Pin_2), R19.1, R25.1, U5.7 (IN1)
- new net VIN_USB: J4.A4 (VBUS), J4.A9 (VBUS), J4.B4 (VBUS), J4.B9 (VBUS)
- no-connect marks 0 -> 3
Other:
- note added: "Does not need external pull ups for D+/- page 179 of datasheet - "USB characteristics""
- note added: "Main battery Can supply pyro rail if pyro battery absent"
- note added: "Pyro supply selection"
- note added: "TODO: check if this PG resistor is actually needed"
- note added: "https://www.digikey.com/en/products/detail/gct/USB4105-GF-A/11198441"
- moved on the sheet: C1, C2, C3, C4, C5, D1, J1, L1, R1, R2, R3, R4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
