File: avionics/avionics_rev1/power_setup.kicad_sch (KiCad schematic)
At the start: 73 parts, among them J1 Conn_01x02, J2 Conn_01x02, J4 USB4105-GF-A, Q1 DMN2056U-7, U1 LMR604063SBRAKRQ1, U13 TPS2121RUXR, U5 TPS2121RUXR, U6 TLV7041DBVR, U7 TMUX1511RSVR

Commit message: adjusted resistor footprints to 0603
Parts:
- R1, R19, R2, R22, R23, R24, R25, R26, R3, R36, R37, R38, R39, R4, R40, R41, R44, R5: footprint Resistor_SMD:R_0402_1005Metric -> Resistor_SMD:R_0603_1608Metric
Changed lines of the file:
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@@
 			)
 		)
-		(property "Footprint" "Resistor_SMD:R_0402_1005Metric"
+		(property "Footprint" "Resistor_SMD:R_0603_1608Metric"
 			(at 210.82 44.45 0)
 			(hide yes)
@@
 			)
 		)
-		(property "Datasheet" "https://yageogroup.com/component-documentation/download/specsheet/RC0402FR-07120RL"
+		(property "Datasheet" ""
 			(at 210.82 44.45 0)
 			(hide yes)
@@
 			)
 		)
-		(property "Footprint" "Resistor_SMD:R_0402_1005Metric"
+		(property "Footprint" "Resistor_SMD:R_0603_1608Metric"
 			(at 377.19 105.41 0)
 			(hide yes)
@@
 		)
 		(property "Tolerance" "1%"
-			(at 377.19 104.77 0)
+			(at 379.222 102.87 90)
 			(show_name no)
 			(do_not_autoplace yes)
@@
 			)
 		)
-		(property "Footprint" "Resistor_SMD:R_0402_1005Metric"
+		(property "Footprint" "Resistor_SMD:R_0603_1608Metric"
 			(at 118.11 133.35 0)
 			(hide yes)
@@
 			)
 		)
-		(property "Datasheet" "https://yageogroup.com/component-documentation/download/specsheet/RC0402FR-0747KL"
+		(property "Datasheet" ""
 			(at 118.11 133.35 0)
 			(hide yes)
@@
 			)
 		)
-		(property "Footprint" "Resistor_SMD:R_0402_1005Metric"
+		(property "Footprint" "Resistor_SMD:R_0603_1608Metric"
 			(at 367.03 110.49 0)
 			(hide yes)
@@
 			)
 		)
-		(property "Footprint" "Resistor_SMD:R_0402_1005Metric"
+		(property "Footprint" "Resistor_SMD:R_0603_1608Metric"
 			(at 364.49 67.31 0)
 			(hide yes)
@@
 			)
 		)
-		(property "Footprint" "Resistor_SMD:R_0402_1005Metric"
+		(property "Footprint" "Resistor_SMD:R_0603_1608Metric"
 			(at 63.5 129.54 0)
 			(hide yes)
@@
 			)
 		)
-		(property "Datasheet" "https://yageogroup.com/component-documentation/download/specsheet/RT0402BRD0718K2L"
+		(property "Datasheet" ""
 			(at 63.5 129.54 0)
 			(hide yes)
@@
 			)
 		)
-		(property "Footprint" "Resistor_SMD:R_0402_1005Metric"
+		(property "Footprint" "Resistor_SMD:R_0603_1608Metric"
 			(at 298.45 43.18 0)
 			(hide yes)
@@
 			)
 		)
-		(property "Footprint" "Resistor_SMD:R_0402_1005Metric"
+		(property "Footprint" "Resistor_SMD:R_0603_1608Metric"
 			(at 113.03 59.69 0)
 			(hide yes)
@@
 			)
 		)
-		(property "Datasheet" "https://www.koaspeer.com/pdfs/RN73R.pdf"
+		(property "Datasheet" ""
 			(at 113.03 59.69 0)
 			(hide yes)
@@
 			)
 		)
-		(property "Footprint" "Resistor_SMD:R_0402_1005Metric"
+		(property "Footprint" "Resistor_SMD:R_0603_1608Metric"
 			(at 71.12 43.18 0)
 			(hide yes)
@@
 			)
 		)
-		(property "Datasheet" "https://yageogroup.com/component-documentation/download/specsheet/RT0402BRD07220KL"
+		(property "Datasheet" ""
 			(at 71.12 43.18 0)
 			(hide yes)
@@
 			)
 		)
-		(property "Footprint" "Resistor_SMD:R_0402_1005Metric"
+		(property "Footprint" "Resistor_SMD:R_0603_1608Metric"
 			(at 298.45 50.8 0)
 			(hide yes)
@@
 			)
 		)
-		(property "Footprint" "Resistor_SMD:R_0402_1005Metric"
+		(property "Footprint" "Resistor_SMD:R_0603_1608Metric"
 			(at 118.11 125.73 0)
 			(hide yes)
@@
 			)
 		)
-		(property "Datasheet" "https://yageogroup.com/component-documentation/download/specsheet/RC0402FR-0747KL"
+		(property "Datasheet" ""
 			(at 118.11 125.73 0)
 			(hide yes)
@@
 			)
 		)
-		(property "Footprint" "Resistor_SMD:R_0402_1005Metric"
+		(property "Footprint" "Resistor_SMD:R_0603_1608Metric"
 			(at 196.85 44.45 0)
 			(hide yes)
@@
 			)
 		)
-		(property "Footprint" "Resistor_SMD:R_0402_1005Metric"
+		(property "Footprint" "Resistor_SMD:R_0603_1608Metric"
 			(at 63.5 137.16 0)
 			(hide yes)
@@
 			)
 		)
-		(property "Datasheet" "https://yageogroup.com/component-documentation/download/specsheet/RT0402BRD0710KL"
+		(property "Datasheet" ""
 			(at 63.5 137.16 0)
 			(hide yes)
@@
 			)
 		)
-		(property "Footprint" "Resistor_SMD:R_0402_1005Metric"
+		(property "Footprint" "Resistor_SMD:R_0603_1608Metric"
 			(at 71.12 53.34 0)
 			(hide yes)
@@
 			)
 		)
-		(property "Datasheet" "https://yageogroup.com/component-documentation/download/specsheet/RT0402BRD0747KL"
+		(property "Datasheet" ""
 			(at 71.12 53.34 0)
 			(hide yes)
@@
 			)
 		)
-		(property "Footprint" "Resistor_SMD:R_0402_1005Metric"
+		(property "Footprint" "Resistor_SMD:R_0603_1608Metric"
 			(at 359.41 93.98 0)
 			(hide yes)
@@
 			)
 		)
-		(property "Datasheet" "https://yageogroup.com/component-documentation/download/specsheet/RC0402FR-0780K6L"
+		(property "Datasheet" ""
 			(at 359.41 93.98 0)
 			(hide yes)
@@
 			)
 		)
-		(property "Footprint" "Resistor_SMD:R_0402_1005Metric"
+		(property "Footprint" "Resistor_SMD:R_0603_1608Metric"
 			(at 283.21 185.42 0)
 			(hide yes)
@@
 			)
 		)
-		(property "Footprint" "Resistor_SMD:R_0402_1005Metric"
+		(property "Footprint" "Resistor_SMD:R_0603_1608Metric"
 			(at 53.34 114.3 0)
 			(hide yes)
@@
 			)
 		)
-		(property "Datasheet" "https://yageogroup.com/component-documentation/download/specsheet/RT0402BRD0710KL"
+		(property "Datasheet" ""
 			(at 53.34 114.3 0)
 			(hide yes)
@@
 			)
 		)
-		(property "Footprint" "Resistor_SMD:R_0402_1005Metric"
+		(property "Footprint" "Resistor_SMD:R_0603_1608Metric"
 			(at 53.34 106.68 0)
 			(hide yes)
@@
 			)
 		)
-		(property "Datasheet" "https://yageogroup.com/component-documentation/download/specsheet/RT0402BRD0720KL"
+		(property "Datasheet" ""
 			(at 53.34 106.68 0)
 			(hide yes)

Commit message: finished updating footprints
Parts:
- C12, C3, C34, C36, C38: footprint Capacitor_SMD:C_0402_1005Metric -> Capacitor_SMD:C_0603_1608Metric; DigiKey https://www.digikey.com/en/products/detail/murata-electroni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 -> https://www.digikey.com/en/products/detail/kemet/C0603C104K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; MPN GRM155R71A104KA01D -> C0603C104K5RACTU; Manufacturer (none) -> KEMET; Voltage 10V -> 50V
- C18, C2: footprint Capacitor_SMD:C_0402_1005Metric -> Capacitor_SMD:C_0603_1608Metric; DigiKey https://www.digikey.com/en/products/detail/murata-electroni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 -> https://www.digikey.com/en/products/detail/kemet/C0603C104K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; MPN GRM155R71H104KE14D -> C0603C104K5RACTU; Manufacturer Murata -> KEMET
- C19, C35, C45, C53, C54, C55: footprint Capacitor_SMD:C_0402_1005Metric -> Capacitor_SMD:C_0603_1608Metric; DigiKey https://www.digikey.com/en/products/detail/murata-electroni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 -> https://www.digikey.com/en/products/detail/yageo/CC0603KRX7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; MPN GRM155R71C103KA01D -> CC0603KRX7R7BB103; Manufacturer (none) -> Yageo
- C31: Manufacturer (none) -> TDK
- J1, J2: value Conn_01x02 -> Wire_Solder_Pads; footprint (none) -> avionics_footprints:WireSolderPads_1x02_3x2mm_P4mm
- R1: DigiKey https://www.digikey.com/en/products/detail/koa-speer-electronics-inc/RN73R1ETTP1522B25/10001056 -> https://www.digikey.com/en/products/detail/koa-speer-electronics-inc/RN73R1JTTD1522B25/10010452; MPN RN73R1ETTP1522B25 -> RN73R1JTTD1522B25; Power 0.0625W -> 0.1W; Voltage 50V -> 75V
- R19: DigiKey https://www.digikey.com/en/products/detail/yageo/RT0402BRD0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 -> https://www.digikey.com/en/products/detail/yageo/RT0603BRD0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; MPN RT0402BRD0720KL -> RT0603BRD0720KL; Power 0.0625W -> 0.1W; Voltage 50V -> 75V
- R2, R41: DigiKey https://www.digikey.com/en/products/detail/yageo/RC0402FR-0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 -> https://www.digikey.com/en/products/detail/yageo/RC0603FR-0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; MPN RC0402FR-07100KL -> RC0603FR-07100KL; Manufacturer (none) -> Yageo; Power 0.063W -> 0.1W; Voltage 50V -> 75V
- R20, R21: footprint Resistor_SMD:R_0402_1005Metric -> Resistor_SMD:R_0603_1608Metric; DigiKey https://www.digikey.com/en/products/detail/yageo/RC0402FR-0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 -> https://www.digikey.com/en/products/detail/yageo/RC0603FR-0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; MPN RC0402FR-075K1L -> RC0603FR-075K1L; Power 0.0625W -> 0.1W; Voltage 50V -> 75V
- R22, R24: DigiKey https://www.digikey.com/en/products/detail/yageo/RT0402BRD0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 -> https://www.digikey.com/en/products/detail/yageo/RT0603BRD0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; MPN RT0402BRD0710KL -> RT0603BRD0710KL; Power 0.0625W -> 0.1W; Voltage 50V -> 75V
- R23: DigiKey https://www.digikey.com/en/products/detail/yageo/RT0402BRD0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 -> https://www.digikey.com/en/products/detail/yageo/RT0603BRD0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; MPN RT0402BRD0718K2L -> RT0603BRD0718K2L; Power 0.0625W -> 0.1W; Voltage 50V -> 75V
- R25, R26: DigiKey https://www.digikey.com/en/products/detail/yageo/RC0402FR-0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 -> https://www.digikey.com/en/products/detail/yageo/RC0603FR-0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; MPN RC0402FR-0747KL -> RC0603FR-0747KL; Power 0.0625W -> 0.1W; Voltage 50V -> 75V
- R27: footprint Resistor_SMD:R_0402_1005Metric -> Resistor_SMD:R_0603_1608Metric; DigiKey https://www.digikey.com/en/products/detail/yageo/RC0402FR-0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 -> https://www.digikey.com/en/products/detail/yageo/RC0603FR-0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; MPN RC0402FR-07100KL -> RC0603FR-07100KL; Manufacturer (none) -> Yageo; Power 0.063W -> 0.1W; Voltage 50V -> 75V
- R28: footprint Resistor_SMD:R_0402_1005Metric -> Resistor_SMD:R_0603_1608Metric; DigiKey https://www.digikey.com/en/products/detail/yageo/RC0402FR-0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 -> https://www.digikey.com/en/products/detail/yageo/RC0603FR-0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; MPN RC0402FR-071KL -> RC0603FR-071KL; Manufacturer (none) -> Yageo; Power 0.063W -> 0.1W; Voltage 50V -> 75V
- R29, R45: footprint Resistor_SMD:R_0402_1005Metric -> Resistor_SMD:R_0603_1608Metric; DigiKey https://www.digikey.com/en/products/detail/yageo/RC0402FR-0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 -> https://www.digikey.com/en/products/detail/yageo/RC0603FR-0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; MPN RC0402FR-0710KL -> RC0603FR-0710KL; Manufacturer (none) -> Yageo; Power (none) -> 0.1W; Voltage 50V -> 75V
- R3: DigiKey https://www.digikey.com/en/products/detail/yageo/RT0402BRD0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 -> https://www.digikey.com/en/products/detail/yageo/RT0603BRD0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; MPN RT0402BRD07220KL -> RT0603BRD07220KL; Power 0.0625W -> 0.1W; Voltage 50V -> 75V
- R30, R32, R42: footprint Resistor_SMD:R_0402_1005Metric -> Resistor_SMD:R_0603_1608Metric; DigiKey https://www.digikey.com/en/products/detail/yageo/RT0402BRD0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 -> https://www.digikey.com/en/products/detail/yageo/RT0603BRD0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; MPN RT0402BRD0749K9L -> RT0603BRD0749K9L; Power 0.0625W -> 0.1W; Voltage 50V -> 75V
- R31, R33, R43: footprint Resistor_SMD:R_0402_1005Metric -> Resistor_SMD:R_0603_1608Metric; DigiKey https://www.digikey.com/en/products/detail/yageo/RT0402BRD0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 -> https://www.digikey.com/en/products/detail/yageo/RT0603BRD0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; MPN RT0402BRD0710KL -> RT0603BRD0710KL; Power 0.0625W -> 0.1W; Voltage 50V -> 75V
- R34: footprint Resistor_SMD:R_0402_1005Metric -> Resistor_SMD:R_0603_1608Metric; DigiKey https://www.digikey.com/en/products/detail/yageo/RC0402FR-0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 -> https://www.digikey.com/en/products/detail/yageo/RC0603FR-0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; MPN RC0402FR-0722K1L -> RC0603FR-0722K1L; Power 0.0625W -> 0.1W; Voltage 50V -> 75V
- R35: footprint Resistor_SMD:R_0402_1005Metric -> Resistor_SMD:R_0603_1608Metric; DigiKey https://www.digikey.com/en/products/detail/yageo/RC0402FR-0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 -> https://www.digikey.com/en/products/detail/yageo/RC0603FR-0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; MPN RC0402FR-0747KL -> RC0603FR-0747KL; Power 0.0625W -> 0.1W; Voltage 50V -> 75V
- R36: DigiKey https://www.digikey.com/en/products/detail/yageo/RC0402FR-0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 -> https://www.digikey.com/en/products/detail/yageo/RC0603FR-0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; MPN RC0402FR-0715KL -> RC0603FR-0715KL; Power 0.0625W -> 0.1W; Voltage 50V -> 75V
- R37, R38, R44: DigiKey https://www.digikey.com/en/products/detail/yageo/RC0402FR-0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 -> https://www.digikey.com/en/products/detail/yageo/RC0603FR-0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; MPN RC0402FR-0710KL -> RC0603FR-0710KL; Manufacturer (none) -> Yageo; Power (none) -> 0.1W; Voltage 50V -> 75V
- R39: DigiKey https://www.digikey.com/en/products/detail/yageo/RC0402FR-0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 -> https://www.digikey.com/en/products/detail/yageo/RC0603FR-0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; MPN RC0402FR-0780K6L -> RC0603FR-0780K6L; Power 0.0625W -> 0.1W; Voltage 50V -> 75V
- R4: DigiKey https://www.digikey.com/en/products/detail/yageo/RT0402BRD0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 -> https://www.digikey.com/en/products/detail/yageo/RT0603BRD0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; MPN RT0402BRD0747KL -> RT0603BRD0747KL; Power 0.0625W -> 0.1W; Voltage 50V -> 75V
- R40: DigiKey https://www.digikey.com/en/products/detail/yageo/RC0402FR-0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 -> https://www.digikey.com/en/products/detail/yageo/RC0603FR-0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; MPN RC0402FR-071KL -> RC0603FR-071KL; Manufacturer (none) -> Yageo; Power 0.063W -> 0.1W; Voltage 50V -> 75V
- R5: DigiKey https://www.digikey.com/en/products/detail/yageo/RC0402FR-0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 -> https://www.digikey.com/en/products/detail/yageo/RC0603FR-0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; MPN RC0402FR-07120RL -> RC0603FR-07120RL; Power 0.0625W -> 0.1W; Voltage 50V -> 75V
Other:
- note added: "U6 Is used as a pyro battery undervoltage protection. When pyro batt falls below ~3.4v, U6 pulls OV1 HIGH, causing IN1 to become an invalid source."
- note removed: "Pyro supply selection"
- moved on the sheet: C1, C12, C16, C17, C18, C19, C2, C3, C35, C38, C4, C5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

Commit message: layout 1
Parts:
- added H1, H2, H3, H4: MountingHole, MountingHole:MountingHole_2.2mm_M2, symbol Mechanical:MountingHole
- C32, C5, TP5, TP6: now not fitted
Connections:
- net PYRO_POWER: now also C17.1
- net VIN_PYRO_BATT: no longer C17.1
Other:
- note added: "TODO: Add fuses to Pyro power channel Add fuses to Logic power channel Figure out max capacitance calculations for USB"
- note removed: "TODO: Add fuses to Pyro power channel Add fuses to Logic power channel"
- moved on the sheet: C18, C19, R32, R33, R35, TP8, TP9
