File: avionics/avionics_rev1/sensors.kicad_sch (KiCad schematic)
At the start: 11 parts, among them U10 LSM6DSV32XTR, U8 LPS22DFTR, U9 ADXL375BCCZ-RL7

Commit message: latest work
Other:
- note added: "IMU"
- moved on the sheet: C25, C26, R11, U10

Commit message: saving work before chat
Other:
- moved on the sheet: C25, C26, R11, U10

Commit message: working on sensors schematics
Parts:
- R10: value 47k -> 10k
Other:
- note added: "Barometer / Altitude Sensor"
- note added: "TODO: Validate schematic for correctness against datasheets Validate pull up/down resistor values where relevant Assign footprints / 3D models to all components Update resistors/capacitors with tolerances/voltages Determine if U9 needs special tantalum capacitors. If so, find a digikey link and make note."
- note removed: "Barometer / Altitude sensor"
- moved on the sheet: C22, C23, C26, R10, R11, R9, U10, U8, U9
