File: avionics/avionics_rev1/sensors.kicad_sch (KiCad schematic)
At the start: 11 parts, among them U10 LSM6DSV32XTR, U8 LPS22DFTR, U9 ADXL375BCCZ-RL7

Commit message: adjusted resistor footprints to 0603
Parts:
- R10, R11, R9: footprint Resistor_SMD:R_0402_1005Metric -> Resistor_SMD:R_0603_1608Metric
Changed lines of the file:
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@@
 			)
 		)
-		(property "Footprint" "Resistor_SMD:R_0402_1005Metric"
+		(property "Footprint" "Resistor_SMD:R_0603_1608Metric"
 			(at 195.58 63.5 0)
 			(hide yes)
@@
 			)
 		)
-		(property "Footprint" "Resistor_SMD:R_0402_1005Metric"
+		(property "Footprint" "Resistor_SMD:R_0603_1608Metric"
 			(at 127 43.18 0)
 			(hide yes)
@@
 			)
 		)
-		(property "Footprint" "Resistor_SMD:R_0402_1005Metric"
+		(property "Footprint" "Resistor_SMD:R_0603_1608Metric"
 			(at 138.43 105.41 0)
 			(hide yes)

Commit message: finished updating footprints
Parts:
- C22, C23, C25, C26: footprint Capacitor_SMD:C_0402_1005Metric -> Capacitor_SMD:C_0603_1608Metric; DigiKey https://www.digikey.com/en/products/detail/murata-electroni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 -> https://www.digikey.com/en/products/detail/kemet/C0603C104K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; MPN GRM155R71A104KA01D -> C0603C104K5RACTU; Manufacturer (none) -> KEMET; Voltage 10V -> 50V
- R10, R11, R9: DigiKey https://www.digikey.com/en/products/detail/yageo/RC0402FR-0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 -> https://www.digikey.com/en/products/detail/yageo/RC0603FR-0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; MPN RC0402FR-0710KL -> RC0603FR-0710KL; Manufacturer (none) -> Yageo; Power 0.05W -> 0.1W; Voltage 50V -> 75V
Changed lines of the file:
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@@
 			)
 		)
-		(property "Datasheet" ""
+		(property "Datasheet" "https://www.yageogroup.com/component-documentation/download/specsheet/RC0603FR-0710KL"
 			(at 195.58 63.5 0)
 			(hide yes)
@@
 			)
 		)
+		(property "Manufacturer" "Yageo"
+			(at 195.58 63.5 0)
+			(hide yes)
+			(show_name no)
+			(do_not_autoplace no)
+			(effects
+				(font
+					(size 1.27 1.27)
+				)
+			)
+		)
 		(property "Tolerance" "1%"
 			(at 193.04 66.6699 0)
@@
 			)
 		)
-		(property "Power" "0.05W"
+		(property "Power" "0.1W"
 			(at 195.58 63.5 0)
 			(hide yes)
@@
 			)
 		)
-		(property "Voltage" "50V"
+		(property "Voltage" "75V"
 			(at 195.58 63.5 0)
 			(hide yes)
@@
 			)
 		)
-		(property "DigiKey" "https://www.digikey.com/en/products/detail/yageo/RC0402FR-0710KL/726523"
+		(property "DigiKey" "https://www.digikey.com/en/products/detail/yageo/RC0603FR-0710KL/726880"
 			(at 0 0 0)
 			(hide yes)
@@
 			)
 		)
-		(property "MPN" "RC0402FR-0710KL"
+		(property "MPN" "RC0603FR-0710KL"
 			(at 0 0 0)
 			(hide yes)
@@
 			)
 		)
-		(property "Footprint" "Capacitor_SMD:C_0402_1005Metric"
+		(property "Footprint" "Capacitor_SMD:C_0603_1608Metric"
 			(at 124.46 123.19 0)
 			(hide yes)
@@
 			)
 		)
-		(property "Datasheet" ""
+		(property "Datasheet" "https://yageogroup.com/content/datasheet/asset/file/KEM_C1002_X7R_SMD"
 			(at 124.46 123.19 0)
 			(hide yes)
@@
 			)
 		)
+		(property "Manufacturer" "KEMET"
+			(at 124.46 123.19 0)
+			(hide yes)
+			(show_name no)
+			(do_not_autoplace no)
+			(effects
+				(font
+					(size 1.27 1.27)
+				)
+			)
+		)
 		(property "Tolerance" "10%"
 			(at 124.46 123.19 0)
@@
 			)
 		)
-		(property "Voltage" "10V"
+		(property "Voltage" "50V"
 			(at 127 126.3535 0)
 			(show_name no)
@@
 			)
 		)
-		(property "DigiKey" "https://www.digikey.com/en/products/detail/murata-electronics/GRM155R71A104KA01D/3845518"
+		(property "DigiKey" "https://www.digikey.com/en/products/detail/kemet/C0603C104K5RACTU/1465623"
 			(at 0 0 0)
 			(hide yes)
@@
 			)
 		)
-		(property "MPN" "GRM155R71A104KA01D"
+		(property "MPN" "C0603C104K5RACTU"
 			(at 0 0 0)
 			(hide yes)
@@
 			)
 		)
-		(property "Footprint" "Capacitor_SMD:C_0402_1005Metric"
+		(property "Footprint" "Capacitor_SMD:C_0603_1608Metric"
 			(at 25.4 119.38 0)
 			(hide yes)
@@
 			)
 		)
-		(property "Datasheet" ""
+		(property "Datasheet" "https://yageogroup.com/content/datasheet/asset/file/KEM_C1002_X7R_SMD"
 			(at 25.4 119.38 0)
 			(hide yes)
@@
 			)
 		)
+		(property "Manufacturer" "KEMET"
+			(at 25.4 119.38 0)
+			(hide yes)
+			(show_name no)
+			(do_not_autoplace no)
+			(effects
+				(font
+					(size 1.27 1.27)
+				)
+			)
+		)
 		(property "Tolerance" "10%"
 			(at 25.4 119.38 0)
@@
 			)
 		)
-		(property "Voltage" "10V"
+		(property "Voltage" "50V"
 			(at 27.94 122.5435 0)
 			(show_name no)
@@
 			)
 		)
-		(property "DigiKey" "https://www.digikey.com/en/products/detail/murata-electronics/GRM155R71A104KA01D/3845518"
+		(property "DigiKey" "https://www.digikey.com/en/products/detail/kemet/C0603C104K5RACTU/1465623"
 			(at 0 0 0)
 			(hide yes)
@@
 			)
 		)
-		(property "MPN" "GRM155R71A104KA01D"
+		(property "MPN" "C0603C104K5RACTU"
 			(at 0 0 0)
 			(hide yes)
@@
 			)
 		)
-		(property "Footprint" "Capacitor_SMD:C_0402_1005Metric"
+		(property "Footprint" "Capacitor_SMD:C_0603_1608Metric"
 			(at 181.61 36.83 0)
 			(hide yes)
@@
 			)
 		)
-		(property "Datasheet" ""
+		(property "Datasheet" "https://yageogroup.com/content/datasheet/asset/file/KEM_C1002_X7R_SMD"
 			(at 181.61 36.83 0)
 			(hide yes)
@@
 			)
 		)
+		(property "Manufacturer" "KEMET"
+			(at 181.61 36.83 0)
+			(hide yes)
+			(show_name no)
+			(do_not_autoplace no)
+			(effects
+				(font
+					(size 1.27 1.27)
+				)
+			)
+		)
 		(property "Tolerance" "10%"
 			(at 181.61 36.83 0)
@@
 			)
 		)
-		(property "Voltage" "10V"
+		(property "Voltage" "50V"
 			(at 184.15 39.9935 0)
 			(show_name no)
@@
 			)
 		)
-		(property "DigiKey" "https://www.digikey.com/en/products/detail/murata-electronics/GRM155R71A104KA01D/3845518"
+		(property "DigiKey" "https://www.digikey.com/en/products/detail/kemet/C0603C104K5RACTU/1465623"
 			(at 0 0 0)
 			(hide yes)
@@
 			)
 		)
-		(property "MPN" "GRM155R71A104KA01D"
+		(property "MPN" "C0603C104K5RACTU"
 			(at 0 0 0)
 			(hide yes)
@@
 			)
 		)
-		(property "Datasheet" ""
+		(property "Datasheet" "https://www.yageogroup.com/component-documentation/download/specsheet/RC0603FR-0710KL"
 			(at 127 43.18 0)
 			(hide yes)
@@
 			)
 		)
+		(property "Manufacturer" "Yageo"
+			(at 127 43.18 0)
+			(hide yes)
+			(show_name no)
+			(do_not_autoplace no)
+			(effects
+				(font
+					(size 1.27 1.27)
+				)
+			)
+		)
 		(property "Tolerance" "1%"
 			(at 124.46 46.3499 0)
@@
 			)
 		)
-		(property "Power" "0.05W"
+		(property "Power" "0.1W"
 			(at 127 43.18 0)
 			(hide yes)
@@
 			)
 		)
-		(property "Voltage" "50V"
+		(property "Voltage" "75V"
 			(at 127 43.18 0)
 			(hide yes)
@@
 			)
 		)
-		(property "DigiKey" "https://www.digikey.com/en/products/detail/yageo/RC0402FR-0710KL/726523"
+		(property "DigiKey" "https://www.digikey.com/en/products/detail/yageo/RC0603FR-0710KL/726880"
 			(at 0 0 0)
 			(hide yes)
@@
 			)
 		)
-		(property "MPN" "RC0402FR-0710KL"
+		(property "MPN" "RC0603FR-0710KL"
 			(at 0 0 0)
 			(hide yes)
@@
 			)
 		)
-		(property "Datasheet" ""
+		(property "Datasheet" "https://www.yageogroup.com/component-documentation/download/specsheet/RC0603FR-0710KL"
 			(at 138.43 105.41 0)
 			(hide yes)
@@
 			)
 		)
+		(property "Manufacturer" "Yageo"
+			(at 138.43 105.41 0)
+			(hide yes)
+			(show_name no)
+			(do_not_autoplace no)
+			(effects
+				(font
+					(size 1.27 1.27)
+				)
+			)
+		)
 		(property "Tolerance" "1%"
 			(at 135.89 108.5799 0)
@@
 			)
 		)
-		(property "Power" "0.05W"
+		(property "Power" "0.1W"
 			(at 138.43 105.41 0)
 			(hide yes)
@@
 			)
 		)
-		(property "Voltage" "50V"
+		(property "Voltage" "75V"
 			(at 138.43 105.41 0)
 			(hide yes)
@@
 			)
 		)
-		(property "DigiKey" "https://www.digikey.com/en/products/detail/yageo/RC0402FR-0710KL/726523"
+		(property "DigiKey" "https://www.digikey.com/en/products/detail/yageo/RC0603FR-0710KL/726880"
 			(at 0 0 0)
 			(hide yes)
@@
 			)
 		)
-		(property "MPN" "RC0402FR-0710KL"
+		(property "MPN" "RC0603FR-0710KL"
 			(at 0 0 0)
 			(hide yes)
@@
 			)
 		)
-		(property "Footprint" "Capacitor_SMD:C_0402_1005Metric"
+		(property "Footprint" "Capacitor_SMD:C_0603_1608Metric"
 			(at 41.91 53.34 0)
 			(hide yes)
@@
 			)
 		)
-		(property "Datasheet" ""
+		(property "Datasheet" "https://yageogroup.com/content/datasheet/asset/file/KEM_C1002_X7R_SMD"
 			(at 41.91 53.34 0)
 			(hide yes)
@@
 			)
 		)
+		(property "Manufacturer" "KEMET"
+			(at 41.91 53.34 0)
+			(hide yes)
+			(show_name no)
+			(do_not_autoplace no)
+			(effects
+				(font
+					(size 1.27 1.27)
+				)
+			)
+		)
 		(property "Tolerance" "10%"
 			(at 41.91 53.34 0)
@@
 			)
 		)
-		(property "Voltage" "10V"
+		(property "Voltage" "50V"
 			(at 39.37 56.5035 0)
 			(show_name no)
@@
 			)
 		)
-		(property "DigiKey" "https://www.digikey.com/en/products/detail/murata-electronics/GRM155R71A104KA01D/3845518"
+		(property "DigiKey" "https://www.digikey.com/en/products/detail/kemet/C0603C104K5RACTU/1465623"
 			(at 0 0 0)
 			(hide yes)
@@
 			)
 		)
-		(property "MPN" "GRM155R71A104KA01D"
+		(property "MPN" "C0603C104K5RACTU"
 			(at 0 0 0)
 			(hide yes)

Commit message: updated todos
Other:
- note added: "TODO: Find replacement sensors that are actually in stock..."
- note removed: "SENSOR DESIGN NOTES 3.3V, 4-wire SPI; keep all CS high at startup. R9-R11: 10k 1% (0.33mA when selected). Place bypass capacitors at each supply pin. U10: mode 1, Qvar/analog hub disabled. C24 follows ADI tantalum recommendation. DigiKey: TAJA105K016RNJ (478-1649-1-ND) https://www.digikey.com/en/products/detail/kyocera-avx/TAJA105K016RNJ/563757"
Changed lines of the file:
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@@
 		)
 	)
-	(text "SENSOR DESIGN NOTES\n3.3V, 4-wire SPI; keep all CS high at startup.\nR9-R11: 10k 1% (0.33mA when selected).\nPlace bypass capacitors at each supply pin.\nU10: mode 1, Qvar/analog hub disabled.\nC24 follows ADI tantalum recommendation.\nDigiKey: TAJA105K016RNJ (478-1649-1-ND)\nhttps://www.digikey.com/en/products/detail/kyocera-avx/TAJA105K016RNJ/563757"
+	(text "TODO:\nFind replacement sensors that \nare actually in stock...\n"
 		(exclude_from_sim no)
 		(at 177.038 105.41 0)
