File: avionics/avionics_rev1/pyro_channels.kicad_sch (KiCad schematic)
At the start: 12 parts, among them J3 Conn_02x04_Top_Bottom, U3 SIS932EDN-T1-GE3, U4 SIS932EDN-T1-GE3

Commit message: working on sensors schematics
Connections:
- net PYRO_3_FET: no longer J3.2 (Pin_2), U4.6
- new net PYRO_4_FET: J3.2 (Pin_2), U4.6
Other:
- note added: "Pyro power good will be determined by MCU before fire command is sent"
- note added: "TODO: overall design review assign footprints for and gate, connector, fets determine resistor values for FETs dividers pick correct FET footprint / part # pick a connector footprint for J3 (small screw terminal)"
- note removed: "TODO: add 1 more and gate to ensure pyro power and MCU power are good"
- note removed: "TODO: assign footprints for and gate, connector, fets determine resistor values for FETs pick correct FET footprint / part #"
Changed lines of the file:
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@@
 	(generator_version "10.0")
 	(paper "A4")
-	(text "TODO: add 1 more and gate to ensure \npyro power and MCU power are good"
+	(text "Pyro power good will be determined by MCU\nbefore fire command is sent"
 		(exclude_from_sim no)
-		(at 19.304 79.756 0)
+		(at 33.528 69.342 0)
 		(effects
 			(font
@@
 		)
 	)
-	(text "TODO: assign footprints for and gate, connector, fets\ndetermine resistor values for FETs\npick correct FET footprint / part #\n"
+	(text "TODO: \noverall design review\nassign footprints for and gate, connector, fets\ndetermine resistor values for FETs dividers\npick correct FET footprint / part #\npick a connector footprint for J3 (small screw terminal) \n"
 		(exclude_from_sim no)
-		(at 112.014 52.578 0)
+		(at 53.34 28.956 0)
 		(effects
 			(font
-				(size 1.27 1.27)
+				(size 2.032 2.032)
+				(thickness 0.4064)
+				(bold yes)
 			)
+			(justify left)
 		)
 	)
@@
 		)
 	)
-	(label "PYRO_3_FET"
+	(label "PYRO_4_FET"
 		(at 177.8 106.68 0)
 		(effects

Commit message: cleaned up schematics after codex work
Parts:
- added C46, C47, C48, C49: 10n / 16V, Capacitor_SMD:C_0402_1005Metric, symbol rocketry_library:GRM155R71C103KA01D
- added C50: 100n / 10V, Capacitor_SMD:C_0402_1005Metric, symbol rocketry_library:GRM155R71A104KA01D
- added R51: 10k 1%, Resistor_SMD:R_0201_0603Metric, symbol Device:R_Small_US
- added U15: TMUX1511RSVR, avionics_footprints:TMUX1511RSVR_RSV16, symbol rocketry_library:TMUX1511RSVR
- R14, R16, R18, R7: value 27k -> 18k; footprint Resistor_SMD:R_0201_0603Metric -> Resistor_SMD:R_0402_1005Metric; symbol Device:R_Small_US -> rocketry_library:RC0402FR-0718KL; DigiKey (none) -> https://www.digikey.com/en/products/detail/yageo/RC0402FR-0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; MPN (none) -> RC0402FR-0718KL; Power (none) -> 0.063W; Tolerance (none) -> 1%; Voltage (none) -> 50V
- R15, R17, R6, R8: footprint Resistor_SMD:R_0201_0603Metric -> Resistor_SMD:R_0402_1005Metric; symbol Device:R_Small_US -> rocketry_library:RC0402FR-07100KL; DigiKey (none) -> https://www.digikey.com/en/products/detail/yageo/RC0402FR-0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; MPN (none) -> RC0402FR-07100KL; Power (none) -> 0.063W; Tolerance (none) -> 1%; Voltage (none) -> 50V
Connections:
- net +3.3V: now also C50.1, U15.16 (VDD)
- net GND: now also C46.2, C47.2, C48.2, C49.2, C50.2, R51.2, U15.8 (GND)
- net PYRO_1_SENS: now also U15.2 (S1)
- net PYRO_2_SENS: now also U15.5 (S2)
- net PYRO_3_SENS: now also U15.10 (S3)
- net PYRO_4_SENS: now also U15.14 (S4)
- new net ADC_PYRO_1: C46.1, U15.3 (D1)
- new net ADC_PYRO_2: C47.1, U15.6 (D2)
- new net ADC_PYRO_3: C48.1, U15.9 (D3)
- new net ADC_PYRO_4: C49.1, U15.13 (D4)
- new net SENSE_EN: R51.1, U15.1 (SEL1), U15.11 (SEL3), U15.15 (SEL4), U15.4 (SEL2)
- no-connect marks 0 -> 2
Other:
- note added: "Individual Pyro Channel Power Control"
- note added: "Pyro sense: powered-off isolation and ADC filtering"
- note added: "SENSE DESIGN NOTES 100k / 18k dividers: 16.8 V -> 2.563 V nominal; 2.607 V at +/-1% worst-case ratio. U15 and U7 use the MCU 3.3 V rail and common SENSE_EN; R44 holds enable low at reset. TMUX1511 powered-off isolation is specified only for signals <=3.6 V; no transient clamp is implied. 10 nF caps at ADC pins; pyro RC ~153 us. Wait >=5 ms after enable and use long ADC acquisition. Sense reads th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"
- moved on the sheet: J3, R14, R15, R16, R17, R18, R6, R7, R8, SN74LVC08AQPWRQ1, U3, U4

Commit message: saving MCU work before using codex
Other:
- note added: "TODO: overall design review assign footprints for and gate, connector, fets determine resistor values for FETs dividers pick correct FET footprint / part # (dual fet) pick a connector footprint for J3 (small screw terminal)"
- note removed: "TODO: overall design review assign footprints for and gate, connector, fets determine resistor values for FETs dividers pick correct FET footprint / part # pick a connector footprint for J3 (small screw terminal)"
Changed lines of the file:
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@@
 		)
 	)
-	(text "TODO: \noverall design review\nassign footprints for and gate, connector, fets\ndetermine resistor values for FETs dividers\npick correct FET footprint / part #\npick a connector footprint for J3 (small screw terminal) \n"
+	(text "TODO: \noverall design review\nassign footprints for and gate, connector, fets\ndetermine resistor values for FETs dividers\npick correct FET footprint / part # (dual fet)\npick a connector footprint for J3 (small screw terminal) \n"
 		(exclude_from_sim no)
 		(at 297.942 65.786 0)

Commit message: fixed ERC errors
Parts:
- C46, C47, C48, C49: value 10n / 16V -> 10n
- C50: value 100n / 10V -> 100n
- R51: value 10k 1% -> 10k; footprint Resistor_SMD:R_0201_0603Metric -> Resistor_SMD:R_0402_1005Metric; symbol Device:R_Small_US -> rocketry_library:RC0402FR-0710KL; DigiKey (none) -> https://www.digikey.com/en/products/detail/yageo/RC0402FR-0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; MPN (none) -> RC0402FR-0710KL; Voltage (none) -> 50V
Changed lines of the file:
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@@
 	(wire
 		(pts
-			(xy 66.04 82.55) (xy 45.72 82.55)
+			(xy 74.93 39.37) (xy 74.93 41.91)
 		)
 		(stroke
@@
 	(wire
 		(pts
-			(xy 165.1 95.25) (xy 167.64 95.25)
+			(xy 66.04 82.55) (xy 45.72 82.55)
 		)
 		(stroke
@@
 	(wire
 		(pts
-			(xy 100.33 168.91) (xy 105.41 168.91)
+			(xy 165.1 95.25) (xy 167.64 95.25)
 		)
 		(stroke
@@
 	(wire
 		(pts
-			(xy 222.25 72.39) (xy 222.25 68.58)
+			(xy 100.33 168.91) (xy 105.41 168.91)
 		)
 		(stroke
@@
 	(wire
 		(pts
-			(xy 74.93 91.44) (xy 74.93 93.98)
+			(xy 222.25 72.39) (xy 222.25 68.58)
 		)
 		(stroke
@@
 	(wire
 		(pts
-			(xy 74.93 39.37) (xy 74.93 41.91)
-		)
-		(stroke
-			(width 0)
-			(type default)
-		)
-	)
-	(wire
-		(pts
 			(xy 31.75 135.89) (xy 31.75 176.53)
 		)
@@
 	(wire
 		(pts
+			(xy 74.93 91.44) (xy 74.93 93.98)
+		)
+		(stroke
+			(width 0)
+			(type default)
+		)
+	)
+	(wire
+		(pts
 			(xy 45.72 73.66) (xy 45.72 64.77)
 		)
@@
 			)
 		)
-		(property "Value" "10n / 16V"
+		(property "Value" "10n"
 			(at 129.54 180.34 0)
 			(show_name no)
@@
 			)
 		)
-		(property "Value" "10n / 16V"
+		(property "Value" "10n"
 			(at 198.12 180.34 0)
 			(show_name no)
@@
 			)
 		)
-		(property "Value" "10n / 16V"
+		(property "Value" "10n"
 			(at 152.4 180.34 0)
 			(show_name no)
@@
 			)
 		)
-		(property "Value" "10n / 16V"
+		(property "Value" "10n"
 			(at 175.26 180.34 0)
 			(show_name no)
@@
 	)
 	(symbol
-		(lib_id "Device:R_Small_US")
+		(lib_id "rocketry_library:RC0402FR-0710KL")
 		(at 54.61 179.07 0)
 		(unit 1)
@@
 			)
 		)
-		(property "Value" "10k 1%"
+		(property "Value" "10k"
 			(at 60.61 180.34 0)
 			(show_name no)
@@
 			)
 		)
-		(property "Footprint" "Resistor_SMD:R_0201_0603Metric"
+		(property "Footprint" "Resistor_SMD:R_0402_1005Metric"
 			(at 54.61 179.07 0)
 			(hide yes)
@@
 			)
 		)
-		(property "Description" ""
+		(property "Description" "Resistor, small US symbol"
 			(at 54.61 179.07 0)
+			(hide yes)
 			(show_name no)
 			(do_not_autoplace no)
@@
 			)
 		)
+		(property "DigiKey" "https://www.digikey.com/en/products/detail/yageo/RC0402FR-0710KL/726523"
+			(at 0 0 0)
+			(hide yes)
+			(show_name no)
+			(do_not_autoplace no)
+			(effects
+				(font
+					(size 1 1)
+				)
+			)
+		)
+		(property "MPN" "RC0402FR-0710KL"
+			(at 0 0 0)
+			(hide yes)
+			(show_name no)
+			(do_not_autoplace no)
+			(effects
+				(font
+					(size 1 1)
+				)
+			)
+		)
+		(property "Voltage" "50V"
+			(at 0 0 0)
+			(hide yes)
+			(show_name no)
+			(do_not_autoplace no)
+			(effects
+				(font
+					(size 1 1)
+				)
+			)
+		)
+		(property "Dielectric" ""
+			(at 0 0 0)
+			(hide yes)
+			(show_name no)
+			(do_not_autoplace no)
+			(effects
+				(font
+					(size 1 1)
+				)
+			)
+		)
 		(pin "2"
 		)
@@
 			)
 		)
-		(property "Value" "100n / 10V"
+		(property "Value" "100n"
 			(at 38.1 180.34 0)
 			(show_name no)
