File: avionics/avionics_rev1/pyro_channels.kicad_sch (KiCad schematic)
At the start: 19 parts, among them J3 Conn_02x04_Top_Bottom, U15 TMUX1511RSVR, U3 SIS932EDN-T1-GE3, U4 SIS932EDN-T1-GE3

Commit message: adjusted resistor footprints to 0603
Parts:
- R14, R15, R16, R17, R18, R51, R6, R7, R8: footprint Resistor_SMD:R_0402_1005Metric -> Resistor_SMD:R_0603_1608Metric
Changed lines of the file:
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@@
 			)
 		)
-		(property "Footprint" "Resistor_SMD:R_0402_1005Metric"
+		(property "Footprint" "Resistor_SMD:R_0603_1608Metric"
 			(at 127 45.72 0)
 			(hide yes)
@@
 			)
 		)
-		(property "Footprint" "Resistor_SMD:R_0402_1005Metric"
+		(property "Footprint" "Resistor_SMD:R_0603_1608Metric"
 			(at 127 81.28 0)
 			(hide yes)
@@
 			)
 		)
-		(property "Footprint" "Resistor_SMD:R_0402_1005Metric"
+		(property "Footprint" "Resistor_SMD:R_0603_1608Metric"
 			(at 172.72 81.28 0)
 			(hide yes)
@@
 			)
 		)
-		(property "Footprint" "Resistor_SMD:R_0402_1005Metric"
+		(property "Footprint" "Resistor_SMD:R_0603_1608Metric"
 			(at 132.08 50.8 0)
 			(hide yes)
@@
 			)
 		)
-		(property "Footprint" "Resistor_SMD:R_0402_1005Metric"
+		(property "Footprint" "Resistor_SMD:R_0603_1608Metric"
 			(at 132.08 86.36 0)
 			(hide yes)
@@
 			)
 		)
-		(property "Footprint" "Resistor_SMD:R_0402_1005Metric"
+		(property "Footprint" "Resistor_SMD:R_0603_1608Metric"
 			(at 177.8 50.8 0)
 			(hide yes)
@@
 			)
 		)
-		(property "Footprint" "Resistor_SMD:R_0402_1005Metric"
+		(property "Footprint" "Resistor_SMD:R_0603_1608Metric"
 			(at 177.8 86.36 0)
 			(hide yes)
@@
 			)
 		)
-		(property "Footprint" "Resistor_SMD:R_0402_1005Metric"
+		(property "Footprint" "Resistor_SMD:R_0603_1608Metric"
 			(at 54.61 179.07 0)
 			(hide yes)
@@
 			)
 		)
-		(property "Footprint" "Resistor_SMD:R_0402_1005Metric"
+		(property "Footprint" "Resistor_SMD:R_0603_1608Metric"
 			(at 172.72 45.72 0)
 			(hide yes)

Commit message: finished updating footprints
Parts:
- C46, C47, C48, C49: footprint Capacitor_SMD:C_0402_1005Metric -> Capacitor_SMD:C_0603_1608Metric; DigiKey https://www.digikey.com/en/products/detail/murata-electroni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 -> https://www.digikey.com/en/products/detail/yageo/CC0603KRX7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; MPN GRM155R71C103KA01D -> CC0603KRX7R7BB103; Manufacturer (none) -> Yageo
- C50: footprint Capacitor_SMD:C_0402_1005Metric -> Capacitor_SMD:C_0603_1608Metric; DigiKey https://www.digikey.com/en/products/detail/murata-electroni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 -> https://www.digikey.com/en/products/detail/kemet/C0603C104K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; MPN GRM155R71A104KA01D -> C0603C104K5RACTU; Manufacturer (none) -> KEMET; Voltage 10V -> 50V
- J3: value Conn_02x04_Top_Bottom -> 1725711; footprint (none) -> avionics_footprints:Phoenix_1725711_MPT_0.5_8_2.54; Current Rating (none) -> 6A; DigiKey (none) -> https://www.digikey.com/en/products/detail/phoenix-contact/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; DigiKey Part Number (none) -> 277-1279-ND; MPN (none) -> 1725711; Manufacturer (none) -> Phoenix Contact; Pitch (none) -> 2.54mm; Position Count (none) -> 8; Wire Gauge (none) -> 26-20 AWG (manufacturer)
- R14, R16, R18, R7: DigiKey https://www.digikey.com/en/products/detail/yageo/RC0402FR-0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 -> https://www.digikey.com/en/products/detail/yageo/RC0603FR-0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; MPN RC0402FR-0718KL -> RC0603FR-0718KL; Manufacturer (none) -> Yageo; Power 0.063W -> 0.1W; Voltage 50V -> 75V
- R15, R17, R6, R8: DigiKey https://www.digikey.com/en/products/detail/yageo/RC0402FR-0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 -> https://www.digikey.com/en/products/detail/yageo/RC0603FR-0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; MPN RC0402FR-07100KL -> RC0603FR-07100KL; Manufacturer (none) -> Yageo; Power 0.063W -> 0.1W; Voltage 50V -> 75V
- R51: DigiKey https://www.digikey.com/en/products/detail/yageo/RC0402FR-0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 -> https://www.digikey.com/en/products/detail/yageo/RC0603FR-0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; MPN RC0402FR-0710KL -> RC0603FR-0710KL; Manufacturer (none) -> Yageo; Power (none) -> 0.1W; Voltage 50V -> 75V
- U16: renamed from SN74LVC08AQPWRQ1; value (none) -> SN74LVC08AWBQARQ1; footprint (none) -> avionics_footprints:SN74LVC08AWBQARQ1_BQA14; DigiKey (none) -> https://www.digikey.com/en/products/detail/texas-instrument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; MPN (none) -> SN74LVC08AWBQARQ1; Manufacturer (none) -> Texas Instruments
Connections:
- net GND: now also U16.15 (EP)
Other:
- note removed: "TODO: overall design review assign footprints for and gate, connector, fets determine resistor values for FETs dividers pick correct FET footprint / part # (dual fet) pick a connector footprint for J3 (small screw terminal)"

Commit message: layout 1
Parts:
- U3, U4: footprint POWERPAK1212-8_VIS -> avionics_footprints:SIS932EDN_PowerPAK1212_8_Dual; DigiKey (none) -> https://www.digikey.com/en/products/detail/vishay-siliconix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; ID Continuous (none) -> 6A package limit; see datasheet thermal conditions; MPN (none) -> SIS932EDN-T1-GE3; Manufacturer (none) -> Vishay Siliconix; Package (none) -> PowerPAK 1212-8 Dual; RDS(on) Max (none) -> 22mOhm at VGS=4.5V; 26mOhm at VGS=2.5V; VDS (none) -> 30V; VGS Absolute Maximum (none) -> +/-12V
Connections:
- net PYRO_1_FET: now also R6.2, U3.7
- net PYRO_2_FET: now also R8.2, U3.5
- net PYRO_3_FET: now also R17.2, U4.7
- net PYRO_4_FET: now also R15.2, U4.5
