File: gpt_context/outputs/power_setup_cleanup/after/power_setup.kicad_sch (KiCad schematic)
At the start: 61 parts, among them J1 Conn_01x02, J2 Conn_01x02, J4 USB_C_Receptacle_USB2.0_16P, Q1 DMN2056U, U1 LMR604063SBRAKRQ1, U13 TPS2121RUXR, U5 TPS2121RUXR, U6 TLV7041DBV, U7 TMUX1511RSVR

Commit message: chat cleanup of schematic
Parts:
- removed C38: 100n, Capacitor_SMD:C_0402_1005Metric, symbol Device:C_Small
- added C37: 100n, Capacitor_SMD:C_0402_1005Metric, symbol Device:C_Small
- R44: value 10k 1% -> 100k 1%
Connections:
- net GND: now also C37.2
- net USB_D+: now also D2.1 (I/O1); no longer D2.6 (I/O4)
- net USB_D-: now also D2.3 (I/O2); no longer D2.4 (I/O3)
- net VIN_USB: now also C37.1
- net at R25.2, R26.1: no longer U5.5 (OV1), U6.1
- net USB_CC1: now reaches J4.A5 (CC1), R21.2
- net USB_CC1: now also D2.4 (I/O3); no longer D2.1 (I/O1)
- net USB_CC2: now reaches J4.B5 (CC2), R20.2
- net USB_CC2: now also D2.6 (I/O4); no longer D2.3 (I/O2)
- new net: U5.5 (OV1), U6.1
Other:
- moved on the sheet: R20, R21
