File: gpt_context/outputs/power_setup_cleanup/after/pyro_channels.kicad_sch (KiCad schematic)
At the start: 12 parts, among them J3 Conn_02x04_Top_Bottom, U3 SIS932EDN-T1-GE3, U4 SIS932EDN-T1-GE3

Commit message: chat cleanup of schematic
Changed lines of the file:
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@@
 	)
 	(global_label "PYRO_3_SENS"
-		(shape output)
+		(shape input)
 		(at 144.78 110.49 0)
 		(fields_autoplaced yes)
@@
 	)
 	(global_label "PYRO_2_SENS"
-		(shape output)
+		(shape input)
 		(at 190.5 74.93 0)
 		(fields_autoplaced yes)
@@
 	)
 	(global_label "PYRO_1_SENS"
-		(shape output)
+		(shape input)
 		(at 144.78 74.93 0)
 		(fields_autoplaced yes)
@@
 	)
 	(global_label "PYRO_4_SENS"
-		(shape output)
+		(shape input)
 		(at 190.5 110.49 0)
 		(fields_autoplaced yes)
@@
 		(dnp no)
 		(property "Reference" "R7"
-			(at 147.32 78.74 0)
+			(at 148.59 80.01 90)
 			(show_name no)
 			(do_not_autoplace no)
@@
 		)
 		(property "Value" "27k"
-			(at 147.32 81.28 0)
+			(at 146.05 80.01 90)
 			(show_name no)
 			(do_not_autoplace no)
@@
 		(dnp no)
 		(property "Reference" "R18"
-			(at 147.32 114.3 0)
+			(at 148.59 115.57 90)
 			(show_name no)
 			(do_not_autoplace no)
@@
 		)
 		(property "Value" "27k"
-			(at 147.32 116.84 0)
+			(at 146.05 115.57 90)
 			(show_name no)
 			(do_not_autoplace no)
@@
 		(dnp no)
 		(property "Reference" "R14"
-			(at 193.04 78.74 0)
+			(at 194.31 80.01 90)
 			(show_name no)
 			(do_not_autoplace no)
@@
 		)
 		(property "Value" "27k"
-			(at 193.04 81.28 0)
+			(at 191.77 80.01 90)
 			(show_name no)
 			(do_not_autoplace no)
@@
 		(dnp no)
 		(property "Reference" "R16"
-			(at 193.04 114.3 0)
+			(at 194.31 115.57 90)
 			(show_name no)
 			(do_not_autoplace no)
@@
 		)
 		(property "Value" "27k"
-			(at 193.04 116.84 0)
-			(show_name no)
-			(do_not_autoplace no)
+			(at 191.77 115.57 90)
+			(show_name no)
+			(do_not_autoplace no)
