File: gpt_context/outputs/power_setup_cleanup/before/power_setup.kicad_sch (KiCad schematic)
At the start: 61 parts, among them J1 Conn_01x02, J2 Conn_01x02, J4 USB_C_Receptacle_USB2.0_16P, Q1 DMN2056U, U1 LMR604063SBRAKRQ1, U13 TPS2121RUXR, U5 TPS2121RUXR, U6 TLV7041DBV, U7 TMUX1511RSVR

Commit message: chat cleanup of schematic
Parts:
- removed C38: 100n, Capacitor_SMD:C_0402_1005Metric, symbol Device:C_Small
- removed D2: USBLC6-4SC6, Package_TO_SOT_SMD:SOT-23-6, symbol Power_Protection:USBLC6-4SC6
- added D2, D3: TODO, Diode_THT:D_DO-201AE_P15.24mm_Horizontal, symbol Diode:1N62xxCA
- C1: value 4.7u -> 4.7uF; footprint Capacitor_SMD:C_0805_2012Metric -> Capacitor_SMD:C_0201_0603Metric; Dielectric X7R -> (none); Voltage 50V -> (none)
- C12: value 100n -> 0.1u; footprint Capacitor_SMD:C_0402_1005Metric -> (none); Dielectric X7R -> (none); Voltage 10V -> (none)
- C16, C17: footprint Capacitor_SMD:C_0805_2012Metric -> (none); Dielectric X7R -> (none); Voltage 35V -> (none)
- C18: value 100n -> 0.1u; footprint Capacitor_SMD:C_0402_1005Metric -> (none); Dielectric X7R -> (none); Voltage 50V -> (none)
- C19: footprint Capacitor_SMD:C_0402_1005Metric -> (none); Dielectric X7R -> (none); Voltage 10V -> (none)
- C2: value 100n -> 0.1uF; footprint Capacitor_SMD:C_0402_1005Metric -> Capacitor_SMD:C_0201_0603Metric; Dielectric X7R -> (none); Voltage 50V -> (none)
- C3: value 100n -> 0.1uF; Dielectric X7R -> (none); Voltage 10V -> (none)
- C31: value 1u -> 1u / 10V; Dielectric X7R -> (none); Voltage 10V -> (none)
- C32, C33: value 10u -> 10u / 35V; Dielectric X7R -> (none); Voltage 35V -> (none)
- C34, C36: value 100n -> 100n / 10V; Dielectric X7R -> (none); Voltage 10V -> (none)
- C35: value 10n -> 10n / 10V; Dielectric X7R -> (none); Voltage 10V -> (none)
- C4: value 4.7u -> 4.7uF; footprint Capacitor_SMD:C_0603_1608Metric -> Capacitor_SMD:C_0201_0603Metric; Dielectric X7R -> (none); Voltage 16V -> (none)
- C5: value 10u -> 10uF; footprint Capacitor_SMD:C_0805_2012Metric -> Capacitor_SMD:C_0201_0603Metric; Dielectric X7R -> (none); Voltage 16V -> (none)
- R1: value 15.2k 1% -> 15.2ohm; Tolerance 1% -> (none)
- R19: value 20k 0.1% -> 20k; Tolerance 0.1% -> (none)
- R2, R27, R41: value 100k 1% -> 100k; Tolerance 1% -> (none)
- R20, R21: value 5.1k 1% -> 5.1k; Tolerance 1% -> (none)
- R22, R24, R31, R33: value 10k 0.1% -> 10k; Tolerance 0.1% -> (none)
- R23: value 18.2k 0.1% -> 18.2k; Tolerance 0.1% -> (none)
- R25, R26, R35: value 47k 1% -> 47k; Tolerance 1% -> (none)
- R28, R40: value 1k 1% -> 1k; Tolerance 1% -> (none)
- R29, R37, R38: value 10k 1% -> 10k; Tolerance 1% -> (none)
- R3: value 220k 0.1% -> 220k; Tolerance 0.1% -> (none)
- R30, R32: value 49.9k 0.1% -> 49.9k; Tolerance 0.1% -> (none)
- R34: value 22.1k 1% -> 22.1k; Tolerance 1% -> (none)
- R36: value 15k 1% -> 15k; Tolerance 1% -> (none)
- R39: value 80.6k 1% -> 80.6k; Tolerance 1% -> (none)
- R4: value 47k 0.1% -> 47k; Tolerance 0.1% -> (none)
- R42, R43: Tolerance 0.1% -> (none)
- R44: value 10k 1% -> 100k; Tolerance 1% -> (none)
- R5: value 120 1% -> 120; Tolerance 1% -> (none)
Connections:
- net GND: now also D2.1 (A1), D3.1 (A1)
- net USB_D+: now also D3.2 (A2)
- net USB_D-: now also D2.2 (A2)
- net at R25.2, R26.1: no longer U5.5 (OV1), U6.1
- new net: U5.5 (OV1), U6.1
Other:
- note added: "V_bat_max = 16.4v (4cell LiPo) V_adc_max = 3.0v Divider ratio = 3.0/16.4 = 0.238 R_bottom = 47k R_top = 47k * ((16.8/3.0) - 1) = 216.2 = 220k"
- note removed: "D2: one SOT-23-6 package; 4 I/O + VBUS ESD. Place D2/C37 at J4; short, wide ground return. Fixed 5 V only; not sustained-overvoltage protection. https://www.st.com/en/protections-and-emi-filters/usblc6-4.html"
- note removed: "VIN_LOGIC sense; not raw battery R3/R4: 220k/47k (ratio 0.1760) 16.8 V -> 2.957 V at SENS_BATT"
- moved on the sheet: R20, R21
