File: gpt_context/outputs/footprint_assignment/before/power_setup.kicad_sch (KiCad schematic)
At the start: 62 parts, among them J1 Conn_01x02, J2 Conn_01x02, J4 USB_C_Receptacle_USB2.0_16P, Q1 DMN2056U-7, U1 LMR604063SBRAKRQ1, U13 TPS2121RUXR, U5 TPS2121RUXR, U6 TLV7041DBVR, U7 TMUX1511RSVR

Commit message: working on sensors schematics
Parts:
- removed R45: 10k 1%, Resistor_SMD:R_0201_0603Metric, symbol Device:R_Small_US
- D1: footprint avionics_footprints:LTST_C170GKT_0805 -> (none); 3D Model Type Generic package -> (none); DigiKey https://www.digikey.com/en/products/detail/liteon/LTST-C170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 -> (none); MPN LTST-C170GKT -> (none)
- D2: footprint avionics_footprints:USBLC6_4SC6_SOT23_6 -> Package_TO_SOT_SMD:SOT-23-6; 3D Model Type Generic package -> (none); DigiKey https://www.digikey.com/en/products/detail/stmicroelectroni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 -> (none)
- D4: value BZT52C4V7-E3-08 -> BZT52Bxx; footprint avionics_footprints:BZT52C4V7_E3_08_SOD123 -> Diode_SMD:D_SOD-123F; 3D Model Type Generic package -> (none); DigiKey https://www.digikey.com/en/products/detail/vishay-general-s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 -> (none); MPN BZT52C4V7-E3-08 -> (none)
- Q1: value DMN2056U-7 -> DMN2056U; footprint avionics_footprints:DMN2056U_7_SOT23 -> Package_TO_SOT_SMD:SOT-23; 3D Model Type Generic package -> (none); DigiKey https://www.digikey.com/en/products/detail/diodes-incorpora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 -> (none); MPN DMN2056U-7 -> (none)
- U1: footprint avionics_footprints:LMR604063SBRAKRQ1_RAK9 -> RAK0009A-MFG; 3D Model Type Manufacturer package -> (none); DigiKey https://www.digikey.com/en/products/detail/texas-instrument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 -> (none); MPN LMR604063SBRAKRQ1 -> (none)
- U13: footprint avionics_footprints:TPS2121RUXR_RUX12 -> Package_DFN_QFN:Texas_VQFN-HR-12_2x2.5mm_P0.5mm; 3D Model Type Manufacturer package -> (none); DigiKey https://www.digikey.com/en/products/detail/texas-instrument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 -> (none); MPN TPS2121RUXR -> (none)
- U5: footprint avionics_footprints:TPS2121RUXR_RUX12 -> RUX0012A; 3D Model Type Manufacturer package -> (none); DigiKey https://www.digikey.com/en/products/detail/texas-instrument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 -> (none); MPN TPS2121RUXR -> (none)
- U6: value TLV7041DBVR -> TLV7041DBV; footprint avionics_footprints:TLV7041DBVR_SOT23_5 -> Package_TO_SOT_SMD:SOT-23-5; 3D Model Type Generic package -> (none); DigiKey https://www.digikey.com/en/products/detail/texas-instrument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 -> (none); MPN TLV7041DBVR -> (none)
- U7: footprint avionics_footprints:TMUX1511RSVR_RSV16 -> RSV0016A-MFG; 3D Model Type Manufacturer package -> (none); DigiKey https://www.digikey.com/en/products/detail/texas-instrument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 -> (none); MPN TMUX1511RSVR -> (none)
Other:
- note added: "TODO: check if this PG resistor is actually needed"
- note removed: "TODO: Add fuses to Pyro power channel Add fuses to Logic power channel"
- company: Matt Schneider -> (none)
- title: Flight Computer Power Distribution -> (none)
- moved on the sheet: C18, C19, R32, R33, R35
