File: gpt_context/outputs/footprint_assignment/staged/power_setup.kicad_sch (KiCad schematic)
At the start: 62 parts, among them J1 Conn_01x02, J2 Conn_01x02, J4 USB_C_Receptacle_USB2.0_16P, Q1 DMN2056U-7, U1 LMR604063SBRAKRQ1, U13 TPS2121RUXR, U5 TPS2121RUXR, U6 TLV7041DBVR, U7 TMUX1511RSVR

Commit message: working on sensors schematics
Parts:
- removed R45: 10k 1%, Resistor_SMD:R_0201_0603Metric, symbol Device:R_Small_US
Other:
- note added: "TODO: check if this PG resistor is actually needed"
- note removed: "TODO: Add fuses to Pyro power channel Add fuses to Logic power channel"
- company: Matt Schneider -> (none)
- title: Flight Computer Power Distribution -> (none)
- moved on the sheet: C18, C19, R32, R33, R35
