File: gpt_context/outputs/sensors_cleanup/before/sensors.kicad_sch (KiCad schematic)
At the start: 11 parts, among them U10 LSM6DSV32XTR, U8 LPS22DFTR, U9 ADXL375BCCZ-RL7

Commit message: updated sensors schematic footprints
Parts:
- C22, C23, C25, C26: value 100n 10% -> 0.1uF; Dielectric X7R -> (none); Tolerance 10% -> (none); Voltage 10V -> (none)
- C24: value 1u 10% -> 1uF; footprint avionics_footprints:TAJA105K016RNJ_3216_18 -> Capacitor_SMD:C_0201_0603Metric; symbol Device:C_Polarized_Small -> Device:C_Small; 3D Model Type KiCad generic 3216-18 package -> (none); Dielectric Tantalum -> (none); DigiKey https://www.digikey.com/en/products/detail/kyocera-avx/TAJA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 -> (none); MPN TAJA105K016RNJ -> (none); Manufacturer KYOCERA AVX -> (none); Tolerance 10% -> (none); Voltage 16V -> (none)
- R10, R11, R9: value 10k 1% -> 10k; Power 0.05W -> (none); Tolerance 1% -> (none); Voltage 25V -> (none)
- U10: footprint avionics_footprints:LGA-14L_2p5X3p0X0p86_STM -> LGA-14L_2p5X3p0X0p86_STM; 3D Model Type Supplier nominal package; visualization only -> (none); MPN LSM6DSV32XTR -> (none)
- U8: footprint avionics_footprints:QFN_22DFTR_STM -> QFN_22DFTR_STM; 3D Model Type Supplier nominal package; visualization only -> (none); MPN LPS22DFTR -> (none)
- U9: footprint avionics_footprints:LGA_CC-14-1_ADI -> LGA_CC-14-1_ADI; 3D Model Type Supplier nominal package; visualization only -> (none); MPN ADXL375BCCZ-RL7 -> (none)
Connections:
- net +3.3V: now also C24.2; no longer C24.1
- net GND: now also C24.1; no longer C24.2
Other:
- note added: "TODO: Validate schematic for correctness against datasheets Validate pull up/down resistor values where relevant Assign footprints / 3D models to all components Update resistors/capacitors with tolerances/voltages Determine if U9 needs special tantalum capacitors. If so, find a digikey link and make note."
- note added: "The datasheet calls for tantalum caps (pg 26) check if this makes a difference between ceramic capacitors"
- note removed: "C24: 1uF tantalum per ADXL375 p.26. TAJA105K016RNJ, 16V, 10%, A case. Positive pin 1 to +3.3V; place at VS."
- note removed: "SENSOR DESIGN NOTES 3.3V, 4-wire SPI; keep all CS high at startup. R9-R11: 10k 1% (0.33mA when selected). Place bypass capacitors at each supply pin. U10: mode 1, Qvar/analog hub disabled. C24 follows ADI tantalum recommendation. DigiKey: TAJA105K016RNJ (478-1649-1-ND) https://www.digikey.com/en/products/detail/kyocera-avx/TAJA105K016RNJ/563757"
