File: gpt_context/outputs/sensors_cleanup/staged/telemetry.kicad_sch (KiCad schematic)
At the start: 11 parts, among them U11 MAX-M10S-00B

Commit message: updated sensors schematic footprints
Other:
- note added: "TODO: update footprints for AE1 FL1 U6 and TP1"
- note removed: "TODO: figure out best antenna solution for 915mhz, if needed, include an SMA port (undesireable) update footprints for AE1 FL1 U6 and TP1 Add voltages/tolerances for all capacitors/resistors Validate schematic against component datasheets"
Changed lines of the file:
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@@
 	(generator_version "10.0")
 	(paper "A4")
-	(text "TODO: \nfigure out best antenna solution for 915mhz,\nif needed, include an SMA port (undesireable)\nupdate footprints for AE1 FL1 U6 and TP1\nAdd voltages/tolerances for all capacitors/resistors\nValidate schematic against component datasheets\n"
+	(text "TODO: update footprints for AE1 FL1 U6 and TP1\n"
 		(exclude_from_sim no)
-		(at 33.274 36.322 0)
+		(at 59.69 40.132 0)
 		(effects
 			(font
-				(size 2.032 2.032)
-				(thickness 0.4064)
-				(bold yes)
+				(size 1.27 1.27)
 			)
 			(justify left)
